Commit message: Refactor namespace handling in minipock URDF
Added a reusable namespace property for the minipock URDF xacro file and replaced hardcoded "minipock" namespaces in the script.

File: urdf/minipock.urdf.xacro (robot description, xacro)
@@ -1,12 +1,15 @@
 <?xml version="1.0"?>
 <robot name="blueboat" xmlns:xacro="http://ros.org/wiki/xacro">
+  <xacro:property name="namespace" value="minipock"/>
   <xacro:include filename="$(find minipock_description)/urdf/minipock_differential_base.xacro"/>
-  <xacro:minipock_base namespace="minipock"/>
+  <xacro:minipock_base namespace="${namespace}"/>
   <!-- motor -->
   <xacro:include filename="$(find minipock_description)/urdf/motor_stepper.xacro"/>
-  <xacro:motor_stepper namespace="minipock" name="stepper_left" x="-0.098" y="0.0" z="-0.034" R="0.0" P="0.0"
+  <xacro:motor_stepper namespace="${namespace}" name="stepper_left" x="-0.098" y="0.0" z="-0.034" R="0.0" P="0.0"
                        Y="${pi/2}" side="1"/>
-  <xacro:motor_stepper namespace="minipock" name="stepper_right" x="0.098" y="0.0" z="-0.034" R="0.0" P="0.0"
+  <xacro:motor_stepper namespace="${namespace}" name="stepper_right" x="0.098" y="0.0" z="-0.034" R="0.0" P="0.0"
                        Y="${-pi/2}" side="-1"/>
+  <xacro:include filename="$(find minipock_description)/urdf/sensors.xacro"/>
+  <xacro:lds_01 namespace="${namespace}" name="lds_01" x="0.0" y="0.0" z="0.079" R="0.0" P="0.0" Y="0.0"/>
   <gazebo>
     <plugin

Commit message: Updated base link names in various URDF and DAE files
The base link name 'namespace_base_link' in multiple files has been changed to 'base_link'. This change was made in order to standardize base link names and ensure compatibility with other predefined robot configurations. Also, the element positions and orientations were adjusted in 'differential_base_alu.dae' for a more realistic robot model representation.

File: urdf/minipock.urdf.xacro (robot description, xacro)
@@ -6,10 +6,10 @@
   <!-- motor -->
   <xacro:include filename="$(find minipock_description)/urdf/motor_stepper.xacro"/>
-  <xacro:motor_stepper namespace="${namespace}" name="stepper_left" x="-0.098" y="0.0" z="-0.034" R="0.0" P="0.0"
-                       Y="${pi/2}" side="1"/>
-  <xacro:motor_stepper namespace="${namespace}" name="stepper_right" x="0.098" y="0.0" z="-0.034" R="0.0" P="0.0"
-                       Y="${-pi/2}" side="-1"/>
+  <xacro:motor_stepper namespace="${namespace}" name="stepper_left" x="0.0" y="0.098" z="-0.034" R="0.0" P="0.0"
+                       Y="0.0" side="1"/>
+  <xacro:motor_stepper namespace="${namespace}" name="stepper_right" x="0.0" y="-0.098" z="-0.034" R="0.0" P="0.0"
+                       Y="${-pi}" side="-1"/>
   <xacro:include filename="$(find minipock_description)/urdf/sensors.xacro"/>
-  <xacro:lds_01 namespace="${namespace}" name="lds_01" x="0.0" y="0.0" z="0.079" R="0.0" P="0.0" Y="0.0"/>
+  <xacro:lds_01 namespace="${namespace}" name="lds_01" x="0.0" y="0.0" z="0.079" R="0.0" P="0.0" Y="${-pi/2}"/>
   <gazebo>
     <plugin
@@ -22,5 +22,5 @@
       <odom_publish_frequency>50</odom_publish_frequency>
       <topic>cmd_vel</topic>
-      <child_frame_id>minipock_base_link</child_frame_id>
+      <child_frame_id>base_link</child_frame_id>
       <frame_id>odom</frame_id>
     </plugin>

File: urdf/minipock_differential_base.xacro (robot description, xacro)
@@ -2,7 +2,7 @@
 <robot name="minipock" xmlns:xacro="http://ros.org/wiki/xacro">
   <xacro:macro name="minipock_base" params="namespace:=minipock">
-    <link name="${namespace}_base_link">
+    <link name="base_link">
       <visual>
-        <origin xyz="0 0 0.0" rpy="${pi/2} 0 0"/>
+        <origin xyz="0 0 0.0" rpy="0 0 0"/>
         <geometry>
           <mesh filename="package://minipock_description/models/differential_base_alu.dae"/>
@@ -89,21 +89,21 @@
     </link>
     <joint name="${namespace}_structure_pla_joint" type="fixed">
-      <origin xyz="0 0 0.0" rpy="0 0 0"/>
-      <parent link="${namespace}_base_link"/>
+      <origin xyz="0 0 0.0" rpy="0 0 ${-pi/2}"/>
+      <parent link="base_link"/>
       <child link="${namespace}_structure_pla_link"/>
     </joint>
     <joint name="${namespace}_structure_pmma_joint" type="fixed">
-      <origin xyz="0 0 0.0" rpy="0 0 0"/>
-      <parent link="${namespace}_base_link"/>
+      <origin xyz="0 0 0.0" rpy="0 0 ${-pi/2}"/>
+      <parent link="base_link"/>
       <child link="${namespace}_structure_pmma_link"/>
     </joint>
     <joint name="${namespace}_structure_misc_joint" type="fixed">
-      <origin xyz="0 0 0.0" rpy="0 0 0"/>
-      <parent link="${namespace}_base_link"/>
+      <origin xyz="0 0 0.0" rpy="0 0 ${-pi/2}"/>
+      <parent link="base_link"/>
       <child link="${namespace}_structure_misc_link"/>
     </joint>
     <joint name="${namespace}_structure_top_joint" type="fixed">
-      <origin xyz="0 0 0.0" rpy="0 0 0"/>
-      <parent link="${namespace}_base_link"/>
+      <origin xyz="0 0 0.0" rpy="0 0 ${-pi/2}"/>
+      <parent link="base_link"/>
       <child link="${namespace}_structure_top_link"/>
     </joint>

File: urdf/motor_stepper.xacro (robot description, xacro)
@@ -42,5 +42,5 @@
     </link>
     <joint name="${name}_joint" type="fixed">
-      <parent link="${namespace}_base_link"/>
+      <parent link="base_link"/>
       <child link="${name}_base_link"/>
       <origin xyz="${x} ${y} ${z}" rpy="${R} ${P} ${Y}"/>

File: urdf/sensors.xacro (robot description, xacro)
@@ -27,5 +27,5 @@
       <limit effort="1000.0" lower="0.0" upper="0" velocity="0"/>
       <origin xyz="${x} ${y} ${z}" rpy="${R} ${P} ${Y}"/>
-      <parent link="${namespace}_base_link"/>
+      <parent link="base_link"/>
       <child link="${name}_link"/>
     </joint>

Commit message: Update STL files for differential and wheel base

File: urdf/minipock.urdf.xacro (robot description, xacro)
@@ -6,7 +6,7 @@
   <!-- motor -->
   <xacro:include filename="$(find minipock_description)/urdf/motor_stepper.xacro"/>
-  <xacro:motor_stepper namespace="${namespace}" name="stepper_left" x="0.0" y="0.098" z="-0.034" R="0.0" P="0.0"
+  <xacro:motor_stepper namespace="${namespace}" name="stepper_left" x="0.0" y="0.133" z="-0.086" R="0.0" P="0.0"
                        Y="0.0" side="1"/>
-  <xacro:motor_stepper namespace="${namespace}" name="stepper_right" x="0.0" y="-0.098" z="-0.034" R="0.0" P="0.0"
+  <xacro:motor_stepper namespace="${namespace}" name="stepper_right" x="0.0" y="-0.133" z="-0.086" R="0.0" P="0.0"
                        Y="${-pi}" side="-1"/>
   <xacro:include filename="$(find minipock_description)/urdf/sensors.xacro"/>

File: urdf/minipock_differential_base.xacro (robot description, xacro)
@@ -47,6 +47,9 @@
         <origin xyz="0 0 0.0" rpy="0 0 0"/>
         <geometry>
-          <mesh filename="package://minipock_description/models/differential_misc.dae"/>
+          <mesh filename="package://minipock_description/models/differential_misc.stl"/>
         </geometry>
+        <material name="6TRON_2">
+          <color rgba="0.27 0.64 0.52 1.0"/>
+      </material>
       </visual>
     </link>

File: urdf/motor_stepper.xacro (robot description, xacro)
@@ -7,9 +7,6 @@
         <origin xyz="0 0 0.0" rpy="${pi/2} 0 0"/>
         <geometry>
-          <mesh filename="package://minipock_description/models/wheel_base.stl"/>
+          <mesh filename="package://minipock_description/models/wheel_base.dae"/>
         </geometry>
-        <material name="6TRON">
-          <color rgba="0.27 0.64 0.52 1.0"/>
-        </material>
       </visual>
       <inertial>
@@ -23,9 +20,6 @@
         <origin xyz="0 -0.073 0" rpy="${pi/2} 0 0"/>
         <geometry>
-          <mesh filename="package://minipock_description/models/wheel_rotative.stl"/>
+          <mesh filename="package://minipock_description/models/wheel_rotative.dae"/>
         </geometry>
-        <material name="black">
-          <color rgba="0.0 0.0 0.0 1.0"/>
-        </material>
       </visual>
       <collision>

Commit message: Update lds_01 sensor position and orientation

File: urdf/minipock.urdf.xacro (robot description, xacro)
@@ -11,5 +11,5 @@
                        Y="${-pi}" side="-1"/>
   <xacro:include filename="$(find minipock_description)/urdf/sensors.xacro"/>
-  <xacro:lds_01 namespace="${namespace}" name="lds_01" x="0.0" y="0.0" z="0.079" R="0.0" P="0.0" Y="${-pi/2}"/>
+  <xacro:lds_01 namespace="${namespace}" name="lds_01" x="0.0" y="0.0" z="0.050" R="0.0" P="0.0" Y="${pi}"/>
   <gazebo>
     <plugin

File: urdf/sensors.xacro (robot description, xacro)
@@ -4,14 +4,11 @@
     <link name="${name}_link">
       <visual name="${name}_visual">
-        <origin xyz="0 0 0" rpy="0 0 0"/>
+        <origin xyz="0 0 0" rpy="${pi/2} 0 0"/>
         <geometry>
-          <mesh filename="package://minipock_description/models/lds.dae" scale="0.001 0.001 0.001"/>
+          <mesh filename="package://minipock_description/models/lds_visual.dae"/>
         </geometry>
-        <material name="black_lidar">
-          <color rgba="0.1 0.1 0.1 1.0"/>
-        </material>
       </visual>
       <collision name="${name}_collision">
-        <origin xyz="0 0 0" rpy="0 0 0"/>
+        <origin xyz="0 0 0.016" rpy="0 0 0"/>
         <geometry>
           <mesh filename="package://minipock_description/models/lds.dae" scale="0.001 0.001 0.001"/>
