Commit message: Add gazebo joint position controller to motor_stepper.xacro
Added a gazebo joint position controller to motor_stepper macro file for better joint control. The module will help manage joint positions in the simulation environment more effectively. Also changed the collision mesh to rectangular and cylinder shapes from STL files, and added a side parameter to the motor macro to differentiate between left and right side motors.

File: urdf/motor_stepper.xacro (robot description, xacro)
@@ -2,5 +2,5 @@
 <robot name="minipock" xmlns:xacro="http://ros.org/wiki/xacro">
   <xacro:macro name="motor_stepper" params="namespace:=minipock name:=stepper_left x:=0.0 y:=0.0 z:=0.0
-				       R:=0.0 P:=0.0 Y:=0.0">
+				       R:=0.0 P:=0.0 Y:=0.0 side:=1">
     <link name="${name}_base_link">
       <visual>
@@ -16,5 +16,5 @@
         <origin xyz="0 0 0.0" rpy="${pi/2} -0 0"/>
         <geometry>
-          <mesh filename="package://minipock_description/models/wheel_base.stl"/>
+          <rectangular size="0.1 0.1 0.1"/>
         </geometry>
       </collision>
@@ -36,7 +36,7 @@
       </visual>
       <collision>
-        <origin xyz="0 -0.073 0" rpy="${pi/2} -0 0"/>
+        <origin xyz="0 ${-0.006/2} 0" rpy="${pi/2} -0 0"/>
         <geometry>
-          <mesh filename="package://minipock_description/models/wheel_rotative.stl"/>
+          <cylinder radius="0.036" length="0.006"/>
         </geometry>
       </collision>
@@ -56,6 +56,16 @@
       <child link="${name}_wheel_link"/>
       <origin xyz="0.0 0.073 0.0" rpy="0 0 0"/>
-      <axis xyz="0 1 0"/>
+      <axis xyz="0 ${side} 0"/>
+      <limit effort="2000" velocity="5"/>
+      <dynamics friction="0.05" damping="0.05"/>
     </joint>
+    <gazebo>
+      <plugin filename="gz-sim-joint-position-controller-system" name="gz::sim::systems::JointPositionController">
+        <joint_name>${name}_wheel_joint</joint_name>
+        <use_velocity_commands>true</use_velocity_commands>
+        <topic>${namespace}/${name}/pos</topic>
+        <name>${name}</name>
+      </plugin>
+    </gazebo>
   </xacro:macro>
 </robot>

Commit message: Fix the geometry of stepper motor in URDF
Changed the URDF geometry config from "rectangular" to "box". The original geometry tag was invalid causing the URDF parser to crash.

File: urdf/motor_stepper.xacro (robot description, xacro)
@@ -16,5 +16,5 @@
         <origin xyz="0 0 0.0" rpy="${pi/2} -0 0"/>
         <geometry>
-          <rectangular size="0.1 0.1 0.1"/>
+          <box size="0.1 0.1 0.1"/>
         </geometry>
       </collision>

Commit message: Remove collision block from motor_stepper
Deleted the collision geometry from the motor_stepper xacro file. This simplifies the representation in the simulator, as the collision block isn't necessary for this component's simulation.

File: urdf/motor_stepper.xacro (robot description, xacro)
@@ -13,10 +13,4 @@
         </material>
       </visual>
-      <collision>
-        <origin xyz="0 0 0.0" rpy="${pi/2} -0 0"/>
-        <geometry>
-          <box size="0.1 0.1 0.1"/>
-        </geometry>
-      </collision>
       <inertial>
         <origin xyz="0.0 -0.029 0.0" rpy="0 -0 0"/>

Commit message: Update motor_stepper.xacro file

File: urdf/motor_stepper.xacro (robot description, xacro)
@@ -1,53 +1,55 @@
 <?xml version="1.0"?>
 <robot name="minipock" xmlns:xacro="http://ros.org/wiki/xacro">
-  <xacro:macro name="motor_stepper" params="namespace:=minipock name:=stepper_left x:=0.0 y:=0.0 z:=0.0
+  <xacro:macro name="motor_stepper"
+    params="namespace:=minipock name:=stepper_left x:=0.0 y:=0.0 z:=0.0
 				       R:=0.0 P:=0.0 Y:=0.0 side:=1">
     <link name="${name}_base_link">
       <visual>
-        <origin xyz="0 0 0.0" rpy="${pi/2} 0 0"/>
+        <origin xyz="0 0 0.0" rpy="${pi/2} 0 0" />
         <geometry>
-          <mesh filename="package://minipock_description/models/wheel_base.dae"/>
+          <mesh filename="package://minipock_description/models/wheel_base.dae" />
         </geometry>
       </visual>
       <inertial>
-        <origin xyz="0.0 -0.029 0.0" rpy="0 -0 0"/>
-        <mass value="1.587"/>
-        <inertia ixx="0.014" ixy="0.0" ixz="0.0" iyy="0.025" iyz="0.0" izz="0.013"/>
+        <origin xyz="0.0 -0.029 0.0" rpy="0 0 0" />
+        <mass value="1.587" />
+        <inertia ixx="0.014" ixy="0.0" ixz="0.0" iyy="0.025" iyz="0.0" izz="0.013" />
       </inertial>
     </link>
     <link name="${name}_wheel_link">
       <visual>
-        <origin xyz="0 -0.073 0" rpy="${pi/2} 0 0"/>
+        <origin xyz="0 0 0" rpy="${pi/2} 0 0" />
         <geometry>
-          <mesh filename="package://minipock_description/models/wheel_rotative.dae"/>
+          <mesh filename="package://minipock_description/models/wheel_rotative.dae" />
         </geometry>
       </visual>
       <collision>
-        <origin xyz="0 ${-0.006/2} 0" rpy="${pi/2} -0 0"/>
+        <origin xyz="0 0.032 0.024" rpy="${pi/2} -0 0" />
         <geometry>
-          <cylinder radius="0.036" length="0.006"/>
+          <cylinder radius="0.036" length="0.006" />
         </geometry>
       </collision>
       <inertial>
-        <origin xyz="0.0 -0.029 0.0" rpy="0 -0 0"/>
-        <mass value="1.587"/>
-        <inertia ixx="0.014" ixy="0.0" ixz="0.0" iyy="0.025" iyz="0.0" izz="0.013"/>
+        <origin xyz="0.0 -0.029 0.0" rpy="0 -0 0" />
+        <mass value="1.587" />
+        <inertia ixx="0.014" ixy="0.0" ixz="0.0" iyy="0.025" iyz="0.0" izz="0.013" />
       </inertial>
     </link>
     <joint name="${name}_joint" type="fixed">
-      <parent link="base_link"/>
-      <child link="${name}_base_link"/>
-      <origin xyz="${x} ${y} ${z}" rpy="${R} ${P} ${Y}"/>
+      <parent link="base_link" />
+      <child link="${name}_base_link" />
+      <origin xyz="${x} ${y} ${z}" rpy="${R} ${P} ${Y}" />
     </joint>
     <joint name="${name}_wheel_joint" type="continuous">
-      <parent link="${name}_base_link"/>
-      <child link="${name}_wheel_link"/>
-      <origin xyz="0.0 0.073 0.0" rpy="0 0 0"/>
-      <axis xyz="0 ${side} 0"/>
-      <limit effort="2000" velocity="5"/>
-      <dynamics friction="0.05" damping="0.05"/>
+      <parent link="${name}_base_link" />
+      <child link="${name}_wheel_link" />
+      <origin xyz="0.0 0.0 0.0" rpy="0 0 0" />
+      <axis xyz="0 ${side} 0" />
+      <limit effort="2000" velocity="5" />
+      <dynamics friction="0.05" damping="0.05" />
     </joint>
     <gazebo>
-      <plugin filename="gz-sim-joint-position-controller-system" name="gz::sim::systems::JointPositionController">
+      <plugin filename="gz-sim-joint-position-controller-system"
+        name="gz::sim::systems::JointPositionController">
         <joint_name>${name}_wheel_joint</joint_name>
         <use_velocity_commands>true</use_velocity_commands>

Commit message: Update motor_stepper.xacro with wheel position and joint origin

File: urdf/motor_stepper.xacro (robot description, xacro)
@@ -19,5 +19,5 @@
     <link name="${name}_wheel_link">
       <visual>
-        <origin xyz="0 0 0" rpy="${pi/2} 0 0" />
+        <origin xyz="0 0 -0.024" rpy="${pi/2} 0 0" />
         <geometry>
           <mesh filename="package://minipock_description/models/wheel_rotative.dae" />
@@ -25,5 +25,5 @@
       </visual>
       <collision>
-        <origin xyz="0 0.032 0.024" rpy="${pi/2} -0 0" />
+        <origin xyz="0 0.032 0.0" rpy="${pi/2} -0 0" />
         <geometry>
           <cylinder radius="0.036" length="0.006" />
@@ -44,5 +44,5 @@
       <parent link="${name}_base_link" />
       <child link="${name}_wheel_link" />
-      <origin xyz="0.0 0.0 0.0" rpy="0 0 0" />
+      <origin xyz="0.0 0.0 0.024" rpy="0 0 0" />
       <axis xyz="0 ${side} 0" />
       <limit effort="2000" velocity="5" />
