Commit message: Update collision geometry and cleanup redundant code
Changed the collision geometry of the mini pock differential base from mesh to a simpler box geometry. This will streamline collision detections and improve performance. Redundant collision entities of various materials were also removed, which contributed to cleaner and more manageable code.

File: urdf/minipock_differential_base.xacro (robot description, xacro)
@@ -10,7 +10,7 @@
       </visual>
       <collision>
-        <origin xyz="0 0 0.0" rpy="${pi/2} -0 0"/>
+        <origin xyz="0 0 -${0.06/2}" rpy="0 -0 0"/>
         <geometry>
-          <mesh filename="package://minipock_description/models/differential_base_alu.dae"/>
+          <box size="0.30 0.342 0.06"/>
         </geometry>
       </collision>
@@ -31,10 +31,4 @@
         </material>
       </visual>
-      <collision>
-        <origin xyz="0 0 0.0" rpy="${pi/2} -0 0"/>
-        <geometry>
-          <mesh filename="package://minipock_description/models/differential_base_pla.stl"/>
-        </geometry>
-      </collision>
       <inertial>
         <origin xyz="0.0 -0.029 0.0" rpy="0 -0 0"/>
@@ -53,10 +47,4 @@
         </material>
       </visual>
-      <collision>
-        <origin xyz="0 0 0.0" rpy="${pi/2} -0 0"/>
-        <geometry>
-          <mesh filename="package://minipock_description/models/differential_base_pmma.stl"/>
-        </geometry>
-      </collision>
       <inertial>
         <origin xyz="0.0 -0.029 0.0" rpy="0 -0 0"/>
@@ -75,10 +63,4 @@
         </material>
       </visual>
-      <collision>
-        <origin xyz="0 0 0.0" rpy="${pi/2} -0 0"/>
-        <geometry>
-          <mesh filename="package://minipock_description/models/differential_misc.stl"/>
-        </geometry>
-      </collision>
       <inertial>
         <origin xyz="0.0 -0.029 0.0" rpy="0 -0 0"/>
@@ -95,5 +77,5 @@
       </visual>
       <collision>
-        <origin xyz="0 0 0.0" rpy="${pi/2} -0 0"/>
+        <origin xyz="0 0 0" rpy="${pi/2} -0 0"/>
         <geometry>
           <mesh filename="package://minipock_description/models/differential_top.dae"/>

Commit message: Increase minipock base size and lidar sensor update rate
The box size for minipock differential base in 'minipock_differential_base.xacro' has been increased for a more accurate representation. Update rate for lidar sensor in 'sensors.xacro' has been increased to improve data capture speed and sensor accuracy.

File: urdf/minipock_differential_base.xacro (robot description, xacro)
@@ -12,5 +12,5 @@
         <origin xyz="0 0 -${0.06/2}" rpy="0 -0 0"/>
         <geometry>
-          <box size="0.30 0.342 0.06"/>
+          <box size="0.30 0.342 0.075"/>
         </geometry>
       </collision>

File: urdf/sensors.xacro (robot description, xacro)
@@ -32,5 +32,5 @@
     <gazebo reference="${name}_link">
       <sensor type="gpu_lidar" name="lds_01">
-        <update_rate>5</update_rate>
+        <update_rate>50</update_rate>
         <topic>scan_raw</topic>
         <visualize>true</visualize>

Commit message: Add Github Actions workflow for ROS2 and simplify URDF model
Created a new Github Actions workflow for building and testing ROS 2 packages automatically upon push and pull request. Also, unnecessary inertial and collision blocks were removed from the minipock_differential_base.xacro URDF model to simplify its structure.

File: urdf/minipock_differential_base.xacro (robot description, xacro)
@@ -31,9 +31,4 @@
         </material>
       </visual>
-      <inertial>
-        <origin xyz="0.0 -0.029 0.0" rpy="0 -0 0"/>
-        <mass value="1.587"/>
-        <inertia ixx="0.014" ixy="0.0" ixz="0.0" iyy="0.025" iyz="0.0" izz="0.013"/>
-      </inertial>
     </link>
     <link name="${namespace}_structure_pmma_link">
@@ -47,9 +42,4 @@
         </material>
       </visual>
-      <inertial>
-        <origin xyz="0.0 -0.029 0.0" rpy="0 -0 0"/>
-        <mass value="1.587"/>
-        <inertia ixx="0.014" ixy="0.0" ixz="0.0" iyy="0.025" iyz="0.0" izz="0.013"/>
-      </inertial>
     </link>
     <link name="${namespace}_structure_misc_link">
@@ -63,9 +53,4 @@
         </material>
       </visual>
-      <inertial>
-        <origin xyz="0.0 -0.029 0.0" rpy="0 -0 0"/>
-        <mass value="1.587"/>
-        <inertia ixx="0.014" ixy="0.0" ixz="0.0" iyy="0.025" iyz="0.0" izz="0.013"/>
-      </inertial>
     </link>
     <link name="${namespace}_structure_top_link">
@@ -76,15 +61,4 @@
         </geometry>
       </visual>
-      <collision>
-        <origin xyz="0 0 0" rpy="${pi/2} -0 0"/>
-        <geometry>
-          <mesh filename="package://minipock_description/models/differential_top.dae"/>
-        </geometry>
-      </collision>
-      <inertial>
-        <origin xyz="0.0 -0.029 0.0" rpy="0 -0 0"/>
-        <mass value="1.587"/>
-        <inertia ixx="0.014" ixy="0.0" ixz="0.0" iyy="0.025" iyz="0.0" izz="0.013"/>
-      </inertial>
     </link>
     <joint name="${namespace}_structure_pla_joint" type="fixed">

Commit message: Update differential base STL files and URDF model

File: urdf/minipock_differential_base.xacro (robot description, xacro)
@@ -4,5 +4,5 @@
     <link name="base_link">
       <visual>
-        <origin xyz="0 0 0.0" rpy="0 0 0"/>
+        <origin xyz="0 0 0.0" rpy="0 0 ${pi/2}"/>
         <geometry>
           <mesh filename="package://minipock_description/models/differential_base_alu.dae"/>
@@ -10,5 +10,5 @@
       </visual>
       <collision>
-        <origin xyz="0 0 -${0.06/2}" rpy="0 -0 0"/>
+        <origin xyz="0 0 -${0.089/2}" rpy="0 -0 ${pi/2}"/>
         <geometry>
           <box size="0.30 0.342 0.075"/>
@@ -23,5 +23,5 @@
     <link name="${namespace}_structure_pla_link">
       <visual>
-        <origin xyz="0 0 0.0" rpy="${pi/2} 0 0"/>
+        <origin xyz="0 0 0.0" rpy="0 0 0"/>
         <geometry>
           <mesh filename="package://minipock_description/models/differential_base_pla.stl"/>
@@ -34,5 +34,5 @@
     <link name="${namespace}_structure_pmma_link">
       <visual>
-        <origin xyz="0 0 0.0" rpy="${pi/2} 0 0"/>
+        <origin xyz="0 0 0.0" rpy="0 0 0"/>
         <geometry>
           <mesh filename="package://minipock_description/models/differential_base_pmma.stl"/>
@@ -45,18 +45,7 @@
     <link name="${namespace}_structure_misc_link">
       <visual>
-        <origin xyz="0 0 0.0" rpy="${pi/2} 0 0"/>
+        <origin xyz="0 0 0.0" rpy="0 0 0"/>
         <geometry>
-          <mesh filename="package://minipock_description/models/differential_misc.stl"/>
-        </geometry>
-        <material name="dark_gray">
-          <color rgba="0.3 0.3 0.3 1.0"/>
-        </material>
-      </visual>
-    </link>
-    <link name="${namespace}_structure_top_link">
-      <visual>
-        <origin xyz="0 0 0.0" rpy="${pi/2} 0 0"/>
-        <geometry>
-          <mesh filename="package://minipock_description/models/differential_top.dae"/>
+          <mesh filename="package://minipock_description/models/differential_misc.dae"/>
         </geometry>
       </visual>
@@ -77,9 +66,4 @@
       <child link="${namespace}_structure_misc_link"/>
     </joint>
-    <joint name="${namespace}_structure_top_joint" type="fixed">
-      <origin xyz="0 0 0.0" rpy="0 0 ${-pi/2}"/>
-      <parent link="base_link"/>
-      <child link="${namespace}_structure_top_link"/>
-    </joint>
   </xacro:macro>
 </robot>

Commit message: Update size of collision box in minipock_differential_base.xacro

File: urdf/minipock_differential_base.xacro (robot description, xacro)
@@ -12,5 +12,5 @@
         <origin xyz="0 0 -${0.089/2}" rpy="0 -0 ${pi/2}"/>
         <geometry>
-          <box size="0.30 0.342 0.075"/>
+          <box size="0.30 0.342 0.089"/>
         </geometry>
       </collision>

Commit message: Update URDF files and Dockerfile

File: urdf/minipock_differential_base.xacro (robot description, xacro)
@@ -4,5 +4,5 @@
     <link name="base_link">
       <visual>
-        <origin xyz="0 0 0.0" rpy="0 0 ${pi/2}"/>
+        <origin xyz="0 0 0.0" rpy="0 0 ${-pi/2}"/>
         <geometry>
           <mesh filename="package://minipock_description/models/differential_base_alu.dae"/>
@@ -10,5 +10,5 @@
       </visual>
       <collision>
-        <origin xyz="0 0 -${0.089/2}" rpy="0 -0 ${pi/2}"/>
+        <origin xyz="0 0 -${0.089/2}" rpy="0 -0 ${-pi/2}"/>
         <geometry>
           <box size="0.30 0.342 0.089"/>
