Commit message: chore: Update generation of multiple robots, better generalization and adding base_footprint concept

File: minipock_description/urdf/minipock_differential_base_v2_b.xacro (robot description, xacro)
@@ -1,5 +1,5 @@
 <?xml version="1.0"?>
 <robot name="minipock" xmlns:xacro="http://ros.org/wiki/xacro">
-  <xacro:macro name="minipock_base" params="namespace:=minipock name:=minipock x:=0 y:=0 z:=0.0">
+  <xacro:macro name="minipock_base" params="namespace:=minipock name:=minipock">
     <link name="${namespace}/base_footprint">
     </link>
@@ -57,5 +57,5 @@
     </link>
     <joint name="base_joint" type="fixed">
-      <origin xyz="${x} ${y} ${z}" rpy="0 0 0"/>
+      <origin xyz="1 0 0.0" rpy="0 0 ${-pi/2}"/>
       <parent link="${namespace}/base_footprint"/>
       <child link="${namespace}/base_link"/>

File: minipock_description/urdf/motor_stepper_v2.xacro (robot description, xacro)
@@ -37,5 +37,5 @@
     </link>
     <joint name="${name}_joint" type="fixed">
-      <parent link="${namespace}/${name}_base_link" />
+      <parent link="${namespace}/base_link" />
       <child link="${namespace}/${name}_base_link" />
       <origin xyz="${x} ${y} ${z}" rpy="${R} ${P} ${Y}" />
