Commit message: feat: cli is used to set the number of robots and the global name of the robots

File: minipock_description/urdf/minipock_differential_base_v2.xacro (robot description, xacro)
@@ -1,8 +1,8 @@
 <?xml version="1.0"?>
 <robot name="minipock" xmlns:xacro="http://ros.org/wiki/xacro">
-  <xacro:macro name="minipock_base" params="namespace:=minipock name:=minipock x:=0 y:=0 z:=0.0">
-    <link name="${namespace}/base_footprint">
+  <xacro:macro name="minipock_base" params="namespace:=minipock/ name:=minipock x:=0 y:=0 z:=0.0">
+    <link name="${namespace}base_footprint">
     </link>
-    <link name="${namespace}/base_link">
+    <link name="${namespace}base_link">
       <visual>
         <origin xyz="0 0 0.0" rpy="0 0 ${-pi/2}"/>
@@ -23,5 +23,5 @@
       </inertial>
     </link>
-    <link name="${namespace}/minipock_structure_pla_link">
+    <link name="${namespace}minipock_structure_pla_link">
       <visual>
         <origin xyz="0 0 0.0" rpy="0 0 0"/>
@@ -34,5 +34,5 @@
       </visual>
     </link>
-    <link name="${namespace}/minipock_structure_pmma_link">
+    <link name="${namespace}minipock_structure_pmma_link">
       <visual>
         <origin xyz="0 0 0.0" rpy="0 0 0"/>
@@ -45,5 +45,5 @@
       </visual>
     </link>
-    <link name="${namespace}/minipock_structure_misc_link">
+    <link name="${namespace}minipock_structure_misc_link">
       <visual>
         <origin xyz="0 0 0.0" rpy="0 0 0"/>
@@ -58,21 +58,21 @@
     <joint name="base_joint" type="fixed">
       <origin xyz="${x} ${y} ${z}" rpy="0 0 0"/>
-      <parent link="${namespace}/base_footprint"/>
-      <child link="${namespace}/base_link"/>
+      <parent link="${namespace}base_footprint"/>
+      <child link="${namespace}base_link"/>
     </joint>
     <joint name="minipock_structure_pla_joint" type="fixed">
       <origin xyz="0 0 0.0" rpy="0 0 ${-pi/2}"/>
-      <parent link="${namespace}/base_link"/>
-      <child link="${namespace}/minipock_structure_pla_link"/>
+      <parent link="${namespace}base_link"/>
+      <child link="${namespace}minipock_structure_pla_link"/>
     </joint>
     <joint name="minipock_structure_pmma_joint" type="fixed">
       <origin xyz="0 0 0.0" rpy="0 0 ${-pi/2}"/>
-      <parent link="${namespace}/base_link"/>
-      <child link="${namespace}/minipock_structure_pmma_link"/>
+      <parent link="${namespace}base_link"/>
+      <child link="${namespace}minipock_structure_pmma_link"/>
     </joint>
     <joint name="minipock_structure_misc_joint" type="fixed">
       <origin xyz="0 0 0.0" rpy="0 0 ${-pi/2}"/>
-      <parent link="${namespace}/base_link"/>
-      <child link="${namespace}/minipock_structure_misc_link"/>
+      <parent link="${namespace}base_link"/>
+      <child link="${namespace}minipock_structure_misc_link"/>
     </joint>
   </xacro:macro>

File: minipock_description/urdf/minipock_v2.urdf.xacro (robot description, xacro)
@@ -1,5 +1,5 @@
 <?xml version="1.0"?>
 <robot name="minipock" xmlns:xacro="http://ros.org/wiki/xacro">
-  <xacro:arg name="namespace" default="minipock"/>
+  <xacro:arg name="namespace" default="minipock/"/>
   <xacro:arg name="x" default="0"/>
   <xacro:arg name="y" default="0"/>
@@ -28,8 +28,8 @@
       <wheel_radius>0.036</wheel_radius>
       <odom_publish_frequency>50</odom_publish_frequency>
-      <topic>${namespace}/cmd_vel</topic>
-      <odom_topic>${namespace}/odom</odom_topic>
-      <child_frame_id>${namespace}/base_footprint</child_frame_id>
-      <frame_id>${namespace}/odom</frame_id>
+      <topic>${namespace}cmd_vel</topic>
+      <odom_topic>${namespace}odom</odom_topic>
+      <child_frame_id>${namespace}base_footprint</child_frame_id>
+      <frame_id>${namespace}odom</frame_id>
     </plugin>
     <plugin filename="libgz-sim-pose-publisher-system.so"

File: minipock_description/urdf/motor_stepper_v2.xacro (robot description, xacro)
@@ -2,7 +2,7 @@
 <robot name="minipock" xmlns:xacro="http://ros.org/wiki/xacro">
   <xacro:macro name="motor_stepper"
-    params="namespace:=minipock name:=stepper_left x:=0.0 y:=0.0 z:=0.0
+    params="namespace:=minipock/ name:=stepper_left x:=0.0 y:=0.0 z:=0.0
 				       R:=0.0 P:=0.0 Y:=0.0 side:=1">
-    <link name="${namespace}/${name}_base_link">
+    <link name="${namespace}${name}_base_link">
       <visual>
         <origin xyz="0 0 0.0" rpy="${pi/2} 0 0" />
@@ -17,5 +17,5 @@
       </inertial>
     </link>
-    <link name="${namespace}/${name}_wheel_link">
+    <link name="${namespace}${name}_wheel_link">
       <visual>
         <origin xyz="0 0 -0.024" rpy="${pi/2} 0 0" />
@@ -37,11 +37,11 @@
     </link>
     <joint name="${name}_joint" type="fixed">
-      <parent link="${namespace}/base_link" />
-      <child link="${namespace}/${name}_base_link" />
+      <parent link="${namespace}base_link" />
+      <child link="${namespace}${name}_base_link" />
       <origin xyz="${x} ${y} ${z}" rpy="${R} ${P} ${Y}" />
     </joint>
     <joint name="${name}_wheel_joint" type="continuous">
-      <parent link="${namespace}/${name}_base_link" />
-      <child link="${namespace}/${name}_wheel_link" />
+      <parent link="${namespace}${name}_base_link" />
+      <child link="${namespace}${name}_wheel_link" />
       <origin xyz="0.0 0.0 0.024" rpy="0 0 0" />
       <axis xyz="0 ${side} 0" />
@@ -54,5 +54,5 @@
         <joint_name>${name}_wheel_joint</joint_name>
         <use_velocity_commands>true</use_velocity_commands>
-        <topic>${namespace}/${name}/pos</topic>
+        <topic>${namespace}${name}/pos</topic>
         <name>${name}</name>
       </plugin>

File: minipock_description/urdf/sensors_v2.xacro (robot description, xacro)
@@ -2,6 +2,6 @@
   <robot name="minipock" xmlns:xacro="http://ros.org/wiki/xacro">
     <xacro:macro name="lds_01"
-                params="namespace:=minipock name:=lds_01 x:=0.0 y:=0.0 z:=0.0 R:=0.0 P:=0.0 Y:=0.0">
-      <link name="${namespace}/${name}_link">
+                params="namespace:=minipock/ name:=lds_01 x:=0.0 y:=0.0 z:=0.0 R:=0.0 P:=0.0 Y:=0.0">
+      <link name="${namespace}${name}_link">
         <visual name="${name}_visual">
           <origin xyz="0 0 0" rpy="${pi/2} 0 0"/>
@@ -25,6 +25,6 @@
         <limit effort="1000.0" lower="0.0" upper="0" velocity="0"/>
         <origin xyz="${x} ${y} ${z}" rpy="${R} ${P} ${Y}"/>
-        <parent link="${namespace}/base_link"/>
-        <child link="${namespace}/${name}_link"/>
+        <parent link="${namespace}base_link"/>
+        <child link="${namespace}${name}_link"/>
       </joint>
       <gazebo reference="${name}_link">
