Commit message: feat: use gz-sim-joint-controller-system plugin for motor.xacro

File: minipock_description/urdf/motor.xacro (robot description, xacro)
@@ -47,9 +47,8 @@
       <axis xyz="0 ${side} 0" />
       <limit effort="2000" velocity="5" />
-      <dynamics friction="0.05" damping="0.05" />
     </joint>
     <gazebo>
-      <plugin filename="gz-sim-joint-position-controller-system"
-        name="gz::sim::systems::JointPositionController">
+      <plugin filename="gz-sim-joint-controller-system"
+        name="gz::sim::systems::JointController">
         <joint_name>${name}_wheel_joint</joint_name>
         <use_velocity_commands>true</use_velocity_commands>

Commit message: feat: Add holonomic wheel option for minipock_description package

File: minipock_description/urdf/motor.xacro (robot description, xacro)
@@ -47,4 +47,13 @@
     <xacro:if value="${mode == 'holonomic'}">
       <link name="${name}_wheel_link">
+        <inertial>
+          <origin
+              xyz="3.3176058353666561185e-10 1.9488714546560112356e-09 -1.4410385216725714439e-09"
+              rpy="0 0 0" />
+          <mass value="0.042007231859596941281" />
+          <inertia ixx="6.621896807313688522e-06" ixy="-3.30985697672957495e-13"
+              ixz="1.2990500681058296834e-10" iyy="1.1099610559885981505e-05"
+              iyz="-7.3482336870196013188e-14" izz="6.6214468781051818449e-06" />
+      </inertial>
         <visual>
           <origin xyz="0 0 0" rpy="0 -0 0" />
@@ -52,43 +61,5 @@
             <mesh filename="package://minipock_description/models/core.stl" />
           </geometry>
-          <material name="core_material">
-            <color
-              rgba="0.91764705882352937127 0.91764705882352937127 0.91764705882352937127 1.0" />
-          </material>
-        </visual>
-        <collision>
-          <origin xyz="0 0 0" rpy="0 -0 0" />
-          <geometry>
-            <mesh filename="package://minipock_description/models/side.stl" />
-          </geometry>
-        </collision>
-        <inertial>
-          <origin xyz="0.0 -0.029 0.0" rpy="0 -0 0" />
-          <mass value="1.587" />
-          <inertia ixx="0.014" ixy="0.0" ixz="0.0" iyy="0.025" iyz="0.0" izz="0.013" />
-        </inertial>
-      </link>
-      <link name="${name}_rollers">
-        <visual>
-          <origin
-            xyz="0.00449999999999999966 -0.019500000000000017319 0.0071250000000000722478"
-            rpy="-3.141592653589793116 -0.52359877559829481886 1.570796326794896558" />
-          <geometry>
-            <mesh filename="package://minipock_description/models/tire.stl" />
-          </geometry>
-        </visual>
-        <collision>
-          <origin
-            xyz="0.00449999999999999966 -0.019500000000000017319 0.0071250000000000722478"
-            rpy="-3.141592653589793116 -0.52359877559829481886 1.570796326794896558" />
-          <geometry>
-            <mesh filename="package://minipock_description/models/tire.stl" />
-          </geometry>
-        </collision>
-        <inertial>
-          <origin xyz="0.0 -0.029 0.0" rpy="0 -0 0" />
-          <mass value="1.587" />
-          <inertia ixx="0.014" ixy="0.0" ixz="0.0" iyy="0.025" iyz="0.0" izz="0.013" />
-        </inertial>
+        </visual>
       </link>
       <joint name="${name}_wheel_joint" type="continuous">
@@ -99,11 +70,391 @@
         <limit effort="2000" velocity="45.5" />
       </joint>
-      <joint name="${name}_continuous_roller_11" type="continuous">
-        <origin xyz="-0.0071249999999999967873 -0.00449999999999999966 0.019500000000000045075"
-          rpy="1.5707963267949005548 -0 1.570796326794896558" />
-        <parent link="${name}_wheel_link" />
-        <child link="${name}_rollers" />
-        <axis xyz="0 0 1" />
-        <limit effort="1" velocity="20" />
+      <link name="${name}_rollers_1">
+        <inertial>
+          <origin xyz="0 0 0" rpy="0 0 0" />
+          <mass value="0.001" />
+          <inertia ixx="0.001" ixy="0" ixz="0" iyy="0.001" iyz="0" izz="0.001" />
+        </inertial>
+        <visual>
+          <origin xyz="0 0 0" rpy="0 -0 0" />
+          <geometry>
+            <mesh filename="package://minipock_description/models/core.stl" />
+          </geometry>
+          <material name="${name}_rollers_1_visual_material">
+            <color
+              rgba="0.91764705882352937127 0.91764705882352937127 0.91764705882352937127 1.0" />
+          </material>
+        </visual>
+      </link>
+      <joint name="${name}_rollers_1_fixing" type="continuous">
+        <origin xyz="0 0 0" rpy="0 -0 0" />
+        <parent link="${name}_wheel_link" />
+        <child link="${name}_rollers_1" />
+        <axis xyz="0 0 1" />
+        <limit effort="1" velocity="20" />
+        <joint_properties friction="0.0" />
+      </joint>
+      <link name="${name}_rollers_2">
+        <inertial>
+          <origin xyz="0 0 0" rpy="0 0 0" />
+          <mass value="0.001" />
+          <inertia ixx="0.001" ixy="0" ixz="0" iyy="0.001" iyz="0" izz="0.001" />
+        </inertial>
+        <visual>
+          <origin xyz="0 0 0"
+            rpy="-3.1696191514317587783e-17 0.52359877559829870464 3.141592653589793116" />
+          <geometry>
+            <mesh filename="package://minipock_description/models/side.stl" />
+          </geometry>
+          <material name="${name}_rollers_2_visual_material">
+            <color rgba="0.2313725490196078538 0.38039215686274507888 0.7058823529411765163 1.0" />
+          </material>
+        </visual>
+      </link>
+      <joint name="${name}_rollers_2_fixing" type="continuous">
+        <origin xyz="0 0 0" rpy="0 -0 0" />
+        <parent link="${name}_wheel_link" />
+        <child link="${name}_rollers_2" />
+        <axis xyz="0 0 1" />
+        <limit effort="1" velocity="20" />
+        <joint_properties friction="0.0" />
+      </joint>
+      <link name="${name}_rollers_3">
+        <inertial>
+          <origin xyz="0 0 0" rpy="0 0 0" />
+          <mass value="0.001" />
+          <inertia ixx="0.001" ixy="0" ixz="0" iyy="0.001" iyz="0" izz="0.001" />
+        </inertial>
+        <visual>
+          <origin xyz="0 0 0" rpy="0 -0 0" />
+          <geometry>
+            <mesh filename="package://minipock_description/models/side.stl" />
+          </geometry>
+          <material name="${name}_rollers_3_visual_material">
+            <color rgba="0.2313725490196078538 0.38039215686274507888 0.7058823529411765163 1.0" />
+          </material>
+        </visual>
+      </link>
+      <joint name="${name}_rollers_3_fixing" type="continuous">
+        <origin xyz="0 0 0" rpy="0 -0 0" />
+        <parent link="${name}_wheel_link" />
+        <child link="${name}_rollers_3" />
+        <axis xyz="0 0 1" />
+        <limit effort="1" velocity="20" />
+        <joint_properties friction="0.0" />
+      </joint>
+      <link name="${name}_rollers_4">
+        <inertial>
+          <origin xyz="0 0 0" rpy="0 0 0" />
+          <mass value="0.001" />
+          <inertia ixx="0.001" ixy="0" ixz="0" iyy="0.001" iyz="0" izz="0.001" />
+        </inertial>
+        <visual>
+          <origin xyz="0 0.00899999999999999932 0"
+            rpy="3.141592653589793116 -0.52359877559829859361 3.141592653589793116" />
+          <geometry>
+            <mesh filename="package://minipock_description/models/tire.stl" />
+          </geometry>
+          <material name="${name}_rollers_4_visual_material">
+            <color
+              rgba="0.49803921568627451677 0.49803921568627451677 0.49803921568627451677 1.0" />
+          </material>
+        </visual>
+      </link>
+      <joint name="${name}_rollers_4_fixing" type="continuous">
+        <origin xyz="0 0 0" rpy="0 -0 0" />
+        <parent link="${name}_wheel_link" />
+        <child link="${name}_rollers_4" />
+        <axis xyz="0 0 1" />
+        <limit effort="1" velocity="20" />
+        <joint_properties friction="0.0" />
+      </joint>
+      <link name="${name}_rollers_5">
+        <inertial>
+          <origin xyz="0 0 0" rpy="0 0 0" />
+          <mass value="0.001" />
+          <inertia ixx="0.001" ixy="0" ixz="0" iyy="0.001" iyz="0" izz="0.001" />
+        </inertial>
+        <visual>
+          <origin xyz="0 0.00899999999999999932 0" rpy="-0 -1.570796326794896558 0" />
+          <geometry>
+            <mesh filename="package://minipock_description/models/tire.stl" />
+          </geometry>
+          <material name="${name}_rollers_5_visual_material">
+            <color
+              rgba="0.49803921568627451677 0.49803921568627451677 0.49803921568627451677 1.0" />
+          </material>
+        </visual>
+      </link>
+      <joint name="${name}_rollers_5_fixing" type="continuous">
+        <origin xyz="0 0 0" rpy="0 -0 0" />
+        <parent link="${name}_wheel_link" />
+        <child link="${name}_rollers_5" />
+        <axis xyz="0 0 1" />
+        <limit effort="1" velocity="20" />
+        <joint_properties friction="0.0" />
+      </joint>
+      <link name="${name}_rollers_6">
+        <inertial>
+          <origin xyz="0 0 0" rpy="0 0 0" />
+          <mass value="0.001" />
+          <inertia ixx="0.001" ixy="0" ixz="0" iyy="0.001" iyz="0" izz="0.001" />
+        </inertial>
+        <visual>
+          <origin xyz="0 0.00899999999999999932 0" rpy="-0 1.570796326794896558 0" />
+          <geometry>
+            <mesh filename="package://minipock_description/models/tire.stl" />
+          </geometry>
+          <material name="${name}_rollers_6_visual_material">
+            <color
+              rgba="0.49803921568627451677 0.49803921568627451677 0.49803921568627451677 1.0" />
+          </material>
+        </visual>
+      </link>
+      <joint name="${name}_rollers_6_fixing" type="continuous">
+        <origin xyz="0 0 0" rpy="0 -0 0" />
+        <parent link="${name}_wheel_link" />
+        <child link="${name}_rollers_6" />
+        <axis xyz="0 0 1" />
+        <limit effort="1" velocity="20" />
+        <joint_properties friction="0.0" />
+      </joint>
+      <link name="${name}_rollers_7">
+        <inertial>
+          <origin xyz="0 0 0" rpy="0 0 0" />
+          <mass value="0.001" />
+          <inertia ixx="0.001" ixy="0" ixz="0" iyy="0.001" iyz="0" izz="0.001" />
+        </inertial>
+        <visual>
+          <origin xyz="0 0.00899999999999999932 0" rpy="0 0.52359877559829870464 0" />
+          <geometry>
+            <mesh filename="package://minipock_description/models/tire.stl" />
+          </geometry>
+          <material name="${name}_rollers_7_visual_material">
+            <color
+              rgba="0.49803921568627451677 0.49803921568627451677 0.49803921568627451677 1.0" />
+          </material>
+        </visual>
+      </link>
+      <joint name="${name}_rollers_7_fixing" type="continuous">
+        <origin xyz="0 0 0" rpy="0 -0 0" />
+        <parent link="${name}_wheel_link" />
+        <child link="${name}_rollers_7" />
+        <axis xyz="0 0 1" />
+        <limit effort="1" velocity="20" />
+        <joint_properties friction="0.0" />
+      </joint>
+      <link name="${name}_rollers_8">
+        <inertial>
+          <origin xyz="0 0 0" rpy="0 0 0" />
+          <mass value="0.001" />
+          <inertia ixx="0.001" ixy="0" ixz="0" iyy="0.001" iyz="0" izz="0.001" />
+        </inertial>
+        <visual>
+          <origin xyz="0 0.00899999999999999932 0" rpy="0 -0.52359877559829914873 0" />
+          <geometry>
+            <mesh filename="package://minipock_description/models/tire.stl" />
+          </geometry>
+          <material name="${name}_rollers_8_visual_material">
+            <color
+              rgba="0.49803921568627451677 0.49803921568627451677 0.49803921568627451677 1.0" />
+          </material>
+        </visual>
+      </link>
+      <joint name="${name}_rollers_8_fixing" type="continuous">
+        <origin xyz="0 0 0" rpy="0 -0 0" />
+        <parent link="${name}_wheel_link" />
+        <child link="${name}_rollers_8" />
+        <axis xyz="0 0 1" />
+        <limit effort="1" velocity="20" />
+        <joint_properties friction="0.0" />
+      </joint>
+      <link name="${name}_rollers_9">
+        <inertial>
+          <origin xyz="0 0 0" rpy="0 0 0" />
+          <mass value="0.001" />
+          <inertia ixx="0.001" ixy="0" ixz="0" iyy="0.001" iyz="0" izz="0.001" />
+        </inertial>
+        <visual>
+          <origin xyz="0 0.00899999999999999932 0"
+            rpy="3.141592653589793116 0.52359877559829914873 3.141592653589793116" />
+          <geometry>
+            <mesh filename="package://minipock_description/models/tire.stl" />
+          </geometry>
+          <material name="${name}_rollers_9_visual_material">
+            <color
+              rgba="0.49803921568627451677 0.49803921568627451677 0.49803921568627451677 1.0" />
+          </material>
+        </visual>
+      </link>
+      <joint name="${name}_rollers_9_fixing" type="continuous">
+        <origin xyz="0 0 0" rpy="0 -0 0" />
+        <parent link="${name}_wheel_link" />
+        <child link="${name}_rollers_9" />
+        <axis xyz="0 0 1" />
+        <limit effort="1" velocity="20" />
+        <joint_properties friction="0.0" />
+      </joint>
+      <link name="${name}_rollers_10">
+        <inertial>
+          <origin xyz="0 0 0" rpy="0 0 0" />
+          <mass value="0.001" />
+          <inertia ixx="0.001" ixy="0" ixz="0" iyy="0.001" iyz="0" izz="0.001" />
+        </inertial>
+        <visual>
+          <origin
+            xyz="2.500000000003367584e-06 -2.7755575615628913511e-17 4.3301270189720353354e-06"
+            rpy="-8.3452360045596450484e-16 -1.0471975511965962991 9.6362485073669450166e-16" />
+          <geometry>
+            <mesh filename="package://minipock_description/models/tire.stl" />
+          </geometry>
+          <material name="${name}_rollers_10_visual_material">
+            <color
+              rgba="0.49803921568627451677 0.49803921568627451677 0.49803921568627451677 1.0" />
+          </material>
+        </visual>
+      </link>
+      <joint name="${name}_rollers_10_fixing" type="continuous">
+        <origin xyz="0 0 0" rpy="0 -0 0" />
+        <parent link="${name}_wheel_link" />
+        <child link="${name}_rollers_10" />
+        <axis xyz="0 0 1" />
+        <limit effort="1" velocity="20" />
+        <joint_properties friction="0.0" />
+      </joint>
+      <link name="${name}_rollers_11">
+        <inertial>
+          <origin xyz="0 0 0" rpy="0 0 0" />
+          <mass value="0.001" />
+          <inertia ixx="0.001" ixy="0" ixz="0" iyy="0.001" iyz="0" izz="0.001" />
+        </inertial>
+        <visual>
+          <origin
+            xyz="-2.5000000000650840986e-06 -1.1265347830754021332e-17 -4.3301270189615499146e-06"
+            rpy="-3.141592653589793116 1.0471975511965965211 3.1415926535897922278" />
+          <geometry>
+            <mesh filename="package://minipock_description/models/tire.stl" />
+          </geometry>
+          <material name="${name}_rollers_11_visual_material">
+            <color
+              rgba="0.49803921568627451677 0.49803921568627451677 0.49803921568627451677 1.0" />
+          </material>
+        </visual>
+      </link>
+      <joint name="${name}_rollers_11_fixing" type="continuous">
+        <origin xyz="0 0 0" rpy="0 -0 0" />
+        <parent link="${name}_wheel_link" />
+        <child link="${name}_rollers_11" />
+        <axis xyz="0 0 1" />
+        <limit effort="1" velocity="20" />
+        <joint_properties friction="0.0" />
+      </joint>
+      <link name="${name}_rollers_12">
+        <inertial>
+          <origin xyz="0 0 0" rpy="0 0 0" />
+          <mass value="0.001" />
+          <inertia ixx="0.001" ixy="0" ixz="0" iyy="0.001" iyz="0" izz="0.001" />
+        </inertial>
+        <visual>
+          <origin
+            xyz="4.9999999999113253768e-06 -2.7755575615628913511e-17 6.9388939039072283776e-18"
+            rpy="1.8722173686805076642e-30 4.3675930115564019462e-15 4.8181242536834853273e-16" />
+          <geometry>
+            <mesh filename="package://minipock_description/models/tire.stl" />
+          </geometry>
+          <material name="${name}_rollers_12_visual_material">
+            <color
+              rgba="0.49803921568627451677 0.49803921568627451677 0.49803921568627451677 1.0" />
+          </material>
+        </visual>
+      </link>
+      <joint name="${name}_rollers_12_fixing" type="continuous">
+        <origin xyz="0 0 0" rpy="0 -0 0" />
+        <parent link="${name}_wheel_link" />
+        <child link="${name}_rollers_12" />
+        <axis xyz="0 0 1" />
+        <limit effort="1" velocity="20" />
+        <joint_properties friction="0.0" />
+      </joint>
+      <link name="${name}_rollers_13">
+        <inertial>
+          <origin xyz="0 0 0" rpy="0 0 0" />
+          <mass value="0.001" />
+          <inertia ixx="0.001" ixy="0" ixz="0" iyy="0.001" iyz="0" izz="0.001" />
+        </inertial>
+        <visual>
+          <origin
+            xyz="-2.5000000000402304579e-06 -2.6888213877640509963e-17 4.3301270189815763145e-06"
+            rpy="-3.1415926535897922278 -1.0471975511965989636 3.1415926535897922278" />
+          <geometry>
+            <mesh filename="package://minipock_description/models/tire.stl" />
+          </geometry>
+          <material name="${name}_rollers_13_visual_material">
+            <color
+              rgba="0.49803921568627451677 0.49803921568627451677 0.49803921568627451677 1.0" />
+          </material>
+        </visual>
+      </link>
+      <joint name="${name}_rollers_13_fixing" type="continuous">
+        <origin xyz="0 0 0" rpy="0 -0 0" />
+        <parent link="${name}_wheel_link" />
+        <child link="${name}_rollers_13" />
+        <axis xyz="0 0 1" />
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