Commit message: feat: Add holonomic wheel option for minipock_description package

File: minipock_description/urdf/motor.xacro (robot description, xacro)
@@ -49,11 +49,11 @@
         <inertial>
           <origin
-              xyz="3.3176058353666561185e-10 1.9488714546560112356e-09 -1.4410385216725714439e-09"
-              rpy="0 0 0" />
+            xyz="3.3176058353666561185e-10 1.9488714546560112356e-09 -1.4410385216725714439e-09"
+            rpy="0 0 0" />
           <mass value="0.042007231859596941281" />
           <inertia ixx="6.621896807313688522e-06" ixy="-3.30985697672957495e-13"
-              ixz="1.2990500681058296834e-10" iyy="1.1099610559885981505e-05"
-              iyz="-7.3482336870196013188e-14" izz="6.6214468781051818449e-06" />
-      </inertial>
+            ixz="1.2990500681058296834e-10" iyy="1.1099610559885981505e-05"
+            iyz="-7.3482336870196013188e-14" izz="6.6214468781051818449e-06" />
+        </inertial>
         <visual>
           <origin xyz="0 0 0" rpy="0 -0 0" />
@@ -61,4 +61,8 @@
             <mesh filename="package://minipock_description/models/core.stl" />
           </geometry>
+          <material name="${name}_rollers_1_visual_material">
+            <color
+              rgba="0.91764705882352937127 0.91764705882352937127 0.91764705882352937127 1.0" />
+          </material>
         </visual>
       </link>
@@ -66,83 +70,14 @@
         <parent link="${name}_base_link" />
         <child link="${name}_wheel_link" />
-        <origin xyz="0.0 0.05 0.024" rpy="0 0 0" />
+        <origin xyz="0.0 0.05 0.0" rpy="0 0 0" />
         <axis xyz="0 ${side} 0" />
         <limit effort="2000" velocity="45.5" />
       </joint>
-      <link name="${name}_rollers_1">
-        <inertial>
-          <origin xyz="0 0 0" rpy="0 0 0" />
-          <mass value="0.001" />
-          <inertia ixx="0.001" ixy="0" ixz="0" iyy="0.001" iyz="0" izz="0.001" />
-        </inertial>
-        <visual>
-          <origin xyz="0 0 0" rpy="0 -0 0" />
-          <geometry>
-            <mesh filename="package://minipock_description/models/core.stl" />
-          </geometry>
-          <material name="${name}_rollers_1_visual_material">
-            <color
-              rgba="0.91764705882352937127 0.91764705882352937127 0.91764705882352937127 1.0" />
-          </material>
-        </visual>
-      </link>
-      <joint name="${name}_rollers_1_fixing" type="continuous">
-        <origin xyz="0 0 0" rpy="0 -0 0" />
-        <parent link="${name}_wheel_link" />
-        <child link="${name}_rollers_1" />
-        <axis xyz="0 0 1" />
-        <limit effort="1" velocity="20" />
-        <joint_properties friction="0.0" />
-      </joint>
-      <link name="${name}_rollers_2">
-        <inertial>
-          <origin xyz="0 0 0" rpy="0 0 0" />
-          <mass value="0.001" />
-          <inertia ixx="0.001" ixy="0" ixz="0" iyy="0.001" iyz="0" izz="0.001" />
-        </inertial>
-        <visual>
-          <origin xyz="0 0 0"
-            rpy="-3.1696191514317587783e-17 0.52359877559829870464 3.141592653589793116" />
-          <geometry>
-            <mesh filename="package://minipock_description/models/side.stl" />
-          </geometry>
-          <material name="${name}_rollers_2_visual_material">
-            <color rgba="0.2313725490196078538 0.38039215686274507888 0.7058823529411765163 1.0" />
-          </material>
-        </visual>
-      </link>
-      <joint name="${name}_rollers_2_fixing" type="continuous">
-        <origin xyz="0 0 0" rpy="0 -0 0" />
-        <parent link="${name}_wheel_link" />
-        <child link="${name}_rollers_2" />
-        <axis xyz="0 0 1" />
-        <limit effort="1" velocity="20" />
-        <joint_properties friction="0.0" />
-      </joint>
-      <link name="${name}_rollers_3">
-        <inertial>
-          <origin xyz="0 0 0" rpy="0 0 0" />
-          <mass value="0.001" />
-          <inertia ixx="0.001" ixy="0" ixz="0" iyy="0.001" iyz="0" izz="0.001" />
-        </inertial>
-        <visual>
-          <origin xyz="0 0 0" rpy="0 -0 0" />
-          <geometry>
-            <mesh filename="package://minipock_description/models/side.stl" />
-          </geometry>
-          <material name="${name}_rollers_3_visual_material">
-            <color rgba="0.2313725490196078538 0.38039215686274507888 0.7058823529411765163 1.0" />
-          </material>
-        </visual>
-      </link>
-      <joint name="${name}_rollers_3_fixing" type="continuous">
-        <origin xyz="0 0 0" rpy="0 -0 0" />
-        <parent link="${name}_wheel_link" />
-        <child link="${name}_rollers_3" />
-        <axis xyz="0 0 1" />
-        <limit effort="1" velocity="20" />
-        <joint_properties friction="0.0" />
-      </joint>
       <link name="${name}_rollers_4">
+        <collision>
+          <geometry>
+            <mesh filename="package://minipock_description/models/tire.stl" />
+          </geometry>
+        </collision>
         <inertial>
           <origin xyz="0 0 0" rpy="0 0 0" />
@@ -168,17 +103,22 @@
         <axis xyz="0 0 1" />
         <limit effort="1" velocity="20" />
-        <joint_properties friction="0.0" />
       </joint>
       <link name="${name}_rollers_5">
-        <inertial>
-          <origin xyz="0 0 0" rpy="0 0 0" />
-          <mass value="0.001" />
-          <inertia ixx="0.001" ixy="0" ixz="0" iyy="0.001" iyz="0" izz="0.001" />
-        </inertial>
-        <visual>
+        <collision>
           <origin xyz="0 0.00899999999999999932 0" rpy="-0 -1.570796326794896558 0" />
           <geometry>
             <mesh filename="package://minipock_description/models/tire.stl" />
           </geometry>
+        </collision>
+        <inertial>
+          <origin xyz="0 0 0" rpy="0 0 0" />
+          <mass value="0.001" />
+          <inertia ixx="0.001" ixy="0" ixz="0" iyy="0.001" iyz="0" izz="0.001" />
+        </inertial>
+        <visual>
+          <origin xyz="0 0.00899999999999999932 0" rpy="-0 -1.570796326794896558 0" />
+          <geometry>
+            <mesh filename="package://minipock_description/models/tire.stl" />
+          </geometry>
           <material name="${name}_rollers_5_visual_material">
             <color
@@ -193,17 +133,22 @@
         <axis xyz="0 0 1" />
         <limit effort="1" velocity="20" />
-        <joint_properties friction="0.0" />
       </joint>
       <link name="${name}_rollers_6">
-        <inertial>
-          <origin xyz="0 0 0" rpy="0 0 0" />
-          <mass value="0.001" />
-          <inertia ixx="0.001" ixy="0" ixz="0" iyy="0.001" iyz="0" izz="0.001" />
-        </inertial>
-        <visual>
+        <collision>
           <origin xyz="0 0.00899999999999999932 0" rpy="-0 1.570796326794896558 0" />
           <geometry>
             <mesh filename="package://minipock_description/models/tire.stl" />
           </geometry>
+        </collision>
+        <inertial>
+          <origin xyz="0 0 0" rpy="0 0 0" />
+          <mass value="0.001" />
+          <inertia ixx="0.001" ixy="0" ixz="0" iyy="0.001" iyz="0" izz="0.001" />
+        </inertial>
+        <visual>
+          <origin xyz="0 0.00899999999999999932 0" rpy="-0 1.570796326794896558 0" />
+          <geometry>
+            <mesh filename="package://minipock_description/models/tire.stl" />
+          </geometry>
           <material name="${name}_rollers_6_visual_material">
             <color
@@ -218,17 +163,22 @@
         <axis xyz="0 0 1" />
         <limit effort="1" velocity="20" />
-        <joint_properties friction="0.0" />
       </joint>
       <link name="${name}_rollers_7">
-        <inertial>
-          <origin xyz="0 0 0" rpy="0 0 0" />
-          <mass value="0.001" />
-          <inertia ixx="0.001" ixy="0" ixz="0" iyy="0.001" iyz="0" izz="0.001" />
-        </inertial>
-        <visual>
+        <collision>
           <origin xyz="0 0.00899999999999999932 0" rpy="0 0.52359877559829870464 0" />
           <geometry>
             <mesh filename="package://minipock_description/models/tire.stl" />
           </geometry>
+        </collision>
+        <inertial>
+          <origin xyz="0 0 0" rpy="0 0 0" />
+          <mass value="0.001" />
+          <inertia ixx="0.001" ixy="0" ixz="0" iyy="0.001" iyz="0" izz="0.001" />
+        </inertial>
+        <visual>
+          <origin xyz="0 0.00899999999999999932 0" rpy="0 0.52359877559829870464 0" />
+          <geometry>
+            <mesh filename="package://minipock_description/models/tire.stl" />
+          </geometry>
           <material name="${name}_rollers_7_visual_material">
             <color
@@ -243,17 +193,22 @@
         <axis xyz="0 0 1" />
         <limit effort="1" velocity="20" />
-        <joint_properties friction="0.0" />
       </joint>
       <link name="${name}_rollers_8">
-        <inertial>
-          <origin xyz="0 0 0" rpy="0 0 0" />
-          <mass value="0.001" />
-          <inertia ixx="0.001" ixy="0" ixz="0" iyy="0.001" iyz="0" izz="0.001" />
-        </inertial>
-        <visual>
+        <collision>
           <origin xyz="0 0.00899999999999999932 0" rpy="0 -0.52359877559829914873 0" />
           <geometry>
             <mesh filename="package://minipock_description/models/tire.stl" />
           </geometry>
+        </collision>
+        <inertial>
+          <origin xyz="0 0 0" rpy="0 0 0" />
+          <mass value="0.001" />
+          <inertia ixx="0.001" ixy="0" ixz="0" iyy="0.001" iyz="0" izz="0.001" />
+        </inertial>
+        <visual>
+          <origin xyz="0 0.00899999999999999932 0" rpy="0 -0.52359877559829914873 0" />
+          <geometry>
+            <mesh filename="package://minipock_description/models/tire.stl" />
+          </geometry>
           <material name="${name}_rollers_8_visual_material">
             <color
@@ -268,13 +223,7 @@
         <axis xyz="0 0 1" />
         <limit effort="1" velocity="20" />
-        <joint_properties friction="0.0" />
       </joint>
       <link name="${name}_rollers_9">
-        <inertial>
-          <origin xyz="0 0 0" rpy="0 0 0" />
-          <mass value="0.001" />
-          <inertia ixx="0.001" ixy="0" ixz="0" iyy="0.001" iyz="0" izz="0.001" />
-        </inertial>
-        <visual>
+        <collision>
           <origin xyz="0 0.00899999999999999932 0"
             rpy="3.141592653589793116 0.52359877559829914873 3.141592653589793116" />
@@ -282,4 +231,16 @@
             <mesh filename="package://minipock_description/models/tire.stl" />
           </geometry>
+        </collision>
+        <inertial>
+          <origin xyz="0 0 0" rpy="0 0 0" />
+          <mass value="0.001" />
+          <inertia ixx="0.001" ixy="0" ixz="0" iyy="0.001" iyz="0" izz="0.001" />
+        </inertial>
+        <visual>
+          <origin xyz="0 0.00899999999999999932 0"
+            rpy="3.141592653589793116 0.52359877559829914873 3.141592653589793116" />
+          <geometry>
+            <mesh filename="package://minipock_description/models/tire.stl" />
+          </geometry>
           <material name="${name}_rollers_9_visual_material">
             <color
@@ -294,13 +255,7 @@
         <axis xyz="0 0 1" />
         <limit effort="1" velocity="20" />
-        <joint_properties friction="0.0" />
       </joint>
       <link name="${name}_rollers_10">
-        <inertial>
-          <origin xyz="0 0 0" rpy="0 0 0" />
-          <mass value="0.001" />
-          <inertia ixx="0.001" ixy="0" ixz="0" iyy="0.001" iyz="0" izz="0.001" />
-        </inertial>
-        <visual>
+        <collision>
           <origin
             xyz="2.500000000003367584e-06 -2.7755575615628913511e-17 4.3301270189720353354e-06"
@@ -309,4 +264,17 @@
             <mesh filename="package://minipock_description/models/tire.stl" />
           </geometry>
+        </collision>
+        <inertial>
+          <origin xyz="0 0 0" rpy="0 0 0" />
+          <mass value="0.001" />
+          <inertia ixx="0.001" ixy="0" ixz="0" iyy="0.001" iyz="0" izz="0.001" />
+        </inertial>
+        <visual>
+          <origin
+            xyz="2.500000000003367584e-06 -2.7755575615628913511e-17 4.3301270189720353354e-06"
+            rpy="-8.3452360045596450484e-16 -1.0471975511965962991 9.6362485073669450166e-16" />
+          <geometry>
+            <mesh filename="package://minipock_description/models/tire.stl" />
+          </geometry>
           <material name="${name}_rollers_10_visual_material">
             <color
@@ -321,13 +289,7 @@
         <axis xyz="0 0 1" />
         <limit effort="1" velocity="20" />
-        <joint_properties friction="0.0" />
       </joint>
       <link name="${name}_rollers_11">
-        <inertial>
-          <origin xyz="0 0 0" rpy="0 0 0" />
-          <mass value="0.001" />
-          <inertia ixx="0.001" ixy="0" ixz="0" iyy="0.001" iyz="0" izz="0.001" />
-        </inertial>
-        <visual>
+        <collision>
           <origin
             xyz="-2.5000000000650840986e-06 -1.1265347830754021332e-17 -4.3301270189615499146e-06"
@@ -336,4 +298,17 @@
             <mesh filename="package://minipock_description/models/tire.stl" />
           </geometry>
+        </collision>
+        <inertial>
+          <origin xyz="0 0 0" rpy="0 0 0" />
+          <mass value="0.001" />
+          <inertia ixx="0.001" ixy="0" ixz="0" iyy="0.001" iyz="0" izz="0.001" />
+        </inertial>
+        <visual>
+          <origin
+            xyz="-2.5000000000650840986e-06 -1.1265347830754021332e-17 -4.3301270189615499146e-06"
+            rpy="-3.141592653589793116 1.0471975511965965211 3.1415926535897922278" />
+          <geometry>
+            <mesh filename="package://minipock_description/models/tire.stl" />
+          </geometry>
           <material name="${name}_rollers_11_visual_material">
             <color
@@ -348,13 +323,7 @@
         <axis xyz="0 0 1" />
         <limit effort="1" velocity="20" />
-        <joint_properties friction="0.0" />
       </joint>
       <link name="${name}_rollers_12">
-        <inertial>
-          <origin xyz="0 0 0" rpy="0 0 0" />
-          <mass value="0.001" />
-          <inertia ixx="0.001" ixy="0" ixz="0" iyy="0.001" iyz="0" izz="0.001" />
-        </inertial>
-        <visual>
+        <collision>
           <origin
             xyz="4.9999999999113253768e-06 -2.7755575615628913511e-17 6.9388939039072283776e-18"
@@ -363,4 +332,17 @@
             <mesh filename="package://minipock_description/models/tire.stl" />
           </geometry>
+        </collision>
+        <inertial>
+          <origin xyz="0 0 0" rpy="0 0 0" />
+          <mass value="0.001" />
+          <inertia ixx="0.001" ixy="0" ixz="0" iyy="0.001" iyz="0" izz="0.001" />
+        </inertial>
+        <visual>
+          <origin
+            xyz="4.9999999999113253768e-06 -2.7755575615628913511e-17 6.9388939039072283776e-18"
+            rpy="1.8722173686805076642e-30 4.3675930115564019462e-15 4.8181242536834853273e-16" />
+          <geometry>
+            <mesh filename="package://minipock_description/models/tire.stl" />
+          </geometry>
           <material name="${name}_rollers_12_visual_material">
             <color
@@ -375,13 +357,7 @@
         <axis xyz="0 0 1" />
         <limit effort="1" velocity="20" />
-        <joint_properties friction="0.0" />
       </joint>
       <link name="${name}_rollers_13">
-        <inertial>
-          <origin xyz="0 0 0" rpy="0 0 0" />
-          <mass value="0.001" />
-          <inertia ixx="0.001" ixy="0" ixz="0" iyy="0.001" iyz="0" izz="0.001" />
-        </inertial>
-        <visual>
+        <collision>
           <origin
             xyz="-2.5000000000402304579e-06 -2.6888213877640509963e-17 4.3301270189815763145e-06"
@@ -390,4 +366,17 @@
             <mesh filename="package://minipock_description/models/tire.stl" />
           </geometry>
+        </collision>
+        <inertial>
+          <origin xyz="0 0 0" rpy="0 0 0" />
+          <mass value="0.001" />
+          <inertia ixx="0.001" ixy="0" ixz="0" iyy="0.001" iyz="0" izz="0.001" />
+        </inertial>
+        <visual>
+          <origin
+            xyz="-2.5000000000402304579e-06 -2.6888213877640509963e-17 4.3301270189815763145e-06"
+            rpy="-3.1415926535897922278 -1.0471975511965989636 3.1415926535897922278" />
+          <geometry>
+            <mesh filename="package://minipock_description/models/tire.stl" />
+          </geometry>
           <material name="${name}_rollers_13_visual_material">
             <color
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