Commit message: feat: Add holonomic wheel option for minipock_description package

File: minipock_description/urdf/motor.xacro (robot description, xacro)
@@ -47,414 +47,327 @@
     <xacro:if value="${mode == 'holonomic'}">
       <link name="${name}_wheel_link">
-        <inertial>
-          <origin
-            xyz="3.3176058353666561185e-10 1.9488714546560112356e-09 -1.4410385216725714439e-09"
-            rpy="0 0 0" />
-          <mass value="0.042007231859596941281" />
-          <inertia ixx="6.621896807313688522e-06" ixy="-3.30985697672957495e-13"
-            ixz="1.2990500681058296834e-10" iyy="1.1099610559885981505e-05"
-            iyz="-7.3482336870196013188e-14" izz="6.6214468781051818449e-06" />
-        </inertial>
-        <visual>
-          <origin xyz="0 0 0" rpy="0 -0 0" />
-          <geometry>
-            <mesh filename="package://minipock_description/models/core.stl" />
-          </geometry>
-          <material name="${name}_rollers_1_visual_material">
-            <color
-              rgba="0.91764705882352937127 0.91764705882352937127 0.91764705882352937127 1.0" />
-          </material>
-        </visual>
+        <visual>
+          <origin xyz="-4.8572257327350598644e-17 0 -0.0099999999999999793915"
+            rpy="1.570796326794896558 -0 -3.8098343924097847915e-13" />
+          <geometry>
+            <mesh filename="package://minipock_description/models/wheel_core.stl" />
+          </geometry>
+          <material name="${name}_wheel_link_material">
+            <color
+              rgba="0.76862745098039220171 0.88627450980392152857 0.95294117647058818044 1.0" />
+          </material>
+        </visual>
+        <inertial>
+          <origin
+            xyz="-7.1267906557384964552e-06 -7.4554367595184111139e-06 -0.0074565222160878352753"
+            rpy="0 0 0" />
+          <mass value="0.0084406729050052354407" />
+          <inertia ixx="1.6585465159980563238e-06" ixy="8.7787669783305516839e-10"
+            ixz="-1.4548784474885956158e-10" iyy="1.6586259130583059041e-06"
+            iyz="-1.5219483721075413049e-10" izz="3.2828932950195218582e-06" />
+        </inertial>
       </link>
       <joint name="${name}_wheel_joint" type="continuous">
         <parent link="${name}_base_link" />
         <child link="${name}_wheel_link" />
-        <origin xyz="0.0 0.05 0.0" rpy="0 0 0" />
-        <axis xyz="0 ${side} 0" />
+        <origin xyz="0.0 0.05 0.024" rpy="${pi/2} 0 0" />
+        <axis xyz="0 0 ${side}" />
         <limit effort="2000" velocity="45.5" />
       </joint>
-      <link name="${name}_rollers_4">
-        <collision>
-          <geometry>
-            <mesh filename="package://minipock_description/models/tire.stl" />
-          </geometry>
-        </collision>
-        <inertial>
-          <origin xyz="0 0 0" rpy="0 0 0" />
-          <mass value="0.001" />
-          <inertia ixx="0.001" ixy="0" ixz="0" iyy="0.001" iyz="0" izz="0.001" />
-        </inertial>
-        <visual>
-          <origin xyz="0 0.00899999999999999932 0"
-            rpy="3.141592653589793116 -0.52359877559829859361 3.141592653589793116" />
-          <geometry>
-            <mesh filename="package://minipock_description/models/tire.stl" />
-          </geometry>
-          <material name="${name}_rollers_4_visual_material">
-            <color
-              rgba="0.49803921568627451677 0.49803921568627451677 0.49803921568627451677 1.0" />
-          </material>
-        </visual>
-      </link>
-      <joint name="${name}_rollers_4_fixing" type="continuous">
-        <origin xyz="0 0 0" rpy="0 -0 0" />
-        <parent link="${name}_wheel_link" />
-        <child link="${name}_rollers_4" />
-        <axis xyz="0 0 1" />
-        <limit effort="1" velocity="20" />
-      </joint>
-      <link name="${name}_rollers_5">
-        <collision>
-          <origin xyz="0 0.00899999999999999932 0" rpy="-0 -1.570796326794896558 0" />
-          <geometry>
-            <mesh filename="package://minipock_description/models/tire.stl" />
-          </geometry>
-        </collision>
-        <inertial>
-          <origin xyz="0 0 0" rpy="0 0 0" />
-          <mass value="0.001" />
-          <inertia ixx="0.001" ixy="0" ixz="0" iyy="0.001" iyz="0" izz="0.001" />
-        </inertial>
-        <visual>
-          <origin xyz="0 0.00899999999999999932 0" rpy="-0 -1.570796326794896558 0" />
-          <geometry>
-            <mesh filename="package://minipock_description/models/tire.stl" />
-          </geometry>
-          <material name="${name}_rollers_5_visual_material">
-            <color
-              rgba="0.49803921568627451677 0.49803921568627451677 0.49803921568627451677 1.0" />
-          </material>
-        </visual>
-      </link>
-      <joint name="${name}_rollers_5_fixing" type="continuous">
-        <origin xyz="0 0 0" rpy="0 -0 0" />
-        <parent link="${name}_wheel_link" />
-        <child link="${name}_rollers_5" />
-        <axis xyz="0 0 1" />
-        <limit effort="1" velocity="20" />
-      </joint>
-      <link name="${name}_rollers_6">
-        <collision>
-          <origin xyz="0 0.00899999999999999932 0" rpy="-0 1.570796326794896558 0" />
-          <geometry>
-            <mesh filename="package://minipock_description/models/tire.stl" />
-          </geometry>
-        </collision>
-        <inertial>
-          <origin xyz="0 0 0" rpy="0 0 0" />
-          <mass value="0.001" />
-          <inertia ixx="0.001" ixy="0" ixz="0" iyy="0.001" iyz="0" izz="0.001" />
-        </inertial>
-        <visual>
-          <origin xyz="0 0.00899999999999999932 0" rpy="-0 1.570796326794896558 0" />
-          <geometry>
-            <mesh filename="package://minipock_description/models/tire.stl" />
-          </geometry>
-          <material name="${name}_rollers_6_visual_material">
-            <color
-              rgba="0.49803921568627451677 0.49803921568627451677 0.49803921568627451677 1.0" />
-          </material>
-        </visual>
-      </link>
-      <joint name="${name}_rollers_6_fixing" type="continuous">
-        <origin xyz="0 0 0" rpy="0 -0 0" />
-        <parent link="${name}_wheel_link" />
-        <child link="${name}_rollers_6" />
-        <axis xyz="0 0 1" />
-        <limit effort="1" velocity="20" />
-      </joint>
-      <link name="${name}_rollers_7">
-        <collision>
-          <origin xyz="0 0.00899999999999999932 0" rpy="0 0.52359877559829870464 0" />
-          <geometry>
-            <mesh filename="package://minipock_description/models/tire.stl" />
-          </geometry>
-        </collision>
-        <inertial>
-          <origin xyz="0 0 0" rpy="0 0 0" />
-          <mass value="0.001" />
-          <inertia ixx="0.001" ixy="0" ixz="0" iyy="0.001" iyz="0" izz="0.001" />
-        </inertial>
-        <visual>
-          <origin xyz="0 0.00899999999999999932 0" rpy="0 0.52359877559829870464 0" />
-          <geometry>
-            <mesh filename="package://minipock_description/models/tire.stl" />
-          </geometry>
-          <material name="${name}_rollers_7_visual_material">
-            <color
-              rgba="0.49803921568627451677 0.49803921568627451677 0.49803921568627451677 1.0" />
-          </material>
-        </visual>
-      </link>
-      <joint name="${name}_rollers_7_fixing" type="continuous">
-        <origin xyz="0 0 0" rpy="0 -0 0" />
-        <parent link="${name}_wheel_link" />
-        <child link="${name}_rollers_7" />
-        <axis xyz="0 0 1" />
-        <limit effort="1" velocity="20" />
-      </joint>
-      <link name="${name}_rollers_8">
-        <collision>
-          <origin xyz="0 0.00899999999999999932 0" rpy="0 -0.52359877559829914873 0" />
-          <geometry>
-            <mesh filename="package://minipock_description/models/tire.stl" />
-          </geometry>
-        </collision>
-        <inertial>
-          <origin xyz="0 0 0" rpy="0 0 0" />
-          <mass value="0.001" />
-          <inertia ixx="0.001" ixy="0" ixz="0" iyy="0.001" iyz="0" izz="0.001" />
-        </inertial>
-        <visual>
-          <origin xyz="0 0.00899999999999999932 0" rpy="0 -0.52359877559829914873 0" />
-          <geometry>
-            <mesh filename="package://minipock_description/models/tire.stl" />
-          </geometry>
-          <material name="${name}_rollers_8_visual_material">
-            <color
-              rgba="0.49803921568627451677 0.49803921568627451677 0.49803921568627451677 1.0" />
-          </material>
-        </visual>
-      </link>
-      <joint name="${name}_rollers_8_fixing" type="continuous">
-        <origin xyz="0 0 0" rpy="0 -0 0" />
-        <parent link="${name}_wheel_link" />
-        <child link="${name}_rollers_8" />
-        <axis xyz="0 0 1" />
-        <limit effort="1" velocity="20" />
-      </joint>
-      <link name="${name}_rollers_9">
-        <collision>
-          <origin xyz="0 0.00899999999999999932 0"
-            rpy="3.141592653589793116 0.52359877559829914873 3.141592653589793116" />
-          <geometry>
-            <mesh filename="package://minipock_description/models/tire.stl" />
-          </geometry>
-        </collision>
-        <inertial>
-          <origin xyz="0 0 0" rpy="0 0 0" />
-          <mass value="0.001" />
-          <inertia ixx="0.001" ixy="0" ixz="0" iyy="0.001" iyz="0" izz="0.001" />
-        </inertial>
-        <visual>
-          <origin xyz="0 0.00899999999999999932 0"
-            rpy="3.141592653589793116 0.52359877559829914873 3.141592653589793116" />
-          <geometry>
-            <mesh filename="package://minipock_description/models/tire.stl" />
-          </geometry>
-          <material name="${name}_rollers_9_visual_material">
-            <color
-              rgba="0.49803921568627451677 0.49803921568627451677 0.49803921568627451677 1.0" />
-          </material>
-        </visual>
-      </link>
-      <joint name="${name}_rollers_9_fixing" type="continuous">
-        <origin xyz="0 0 0" rpy="0 -0 0" />
-        <parent link="${name}_wheel_link" />
-        <child link="${name}_rollers_9" />
-        <axis xyz="0 0 1" />
-        <limit effort="1" velocity="20" />
-      </joint>
-      <link name="${name}_rollers_10">
-        <collision>
-          <origin
-            xyz="2.500000000003367584e-06 -2.7755575615628913511e-17 4.3301270189720353354e-06"
-            rpy="-8.3452360045596450484e-16 -1.0471975511965962991 9.6362485073669450166e-16" />
-          <geometry>
-            <mesh filename="package://minipock_description/models/tire.stl" />
-          </geometry>
-        </collision>
-        <inertial>
-          <origin xyz="0 0 0" rpy="0 0 0" />
-          <mass value="0.001" />
-          <inertia ixx="0.001" ixy="0" ixz="0" iyy="0.001" iyz="0" izz="0.001" />
-        </inertial>
-        <visual>
-          <origin
-            xyz="2.500000000003367584e-06 -2.7755575615628913511e-17 4.3301270189720353354e-06"
-            rpy="-8.3452360045596450484e-16 -1.0471975511965962991 9.6362485073669450166e-16" />
-          <geometry>
-            <mesh filename="package://minipock_description/models/tire.stl" />
-          </geometry>
-          <material name="${name}_rollers_10_visual_material">
-            <color
-              rgba="0.49803921568627451677 0.49803921568627451677 0.49803921568627451677 1.0" />
-          </material>
-        </visual>
-      </link>
-      <joint name="${name}_rollers_10_fixing" type="continuous">
-        <origin xyz="0 0 0" rpy="0 -0 0" />
-        <parent link="${name}_wheel_link" />
-        <child link="${name}_rollers_10" />
-        <axis xyz="0 0 1" />
-        <limit effort="1" velocity="20" />
-      </joint>
-      <link name="${name}_rollers_11">
-        <collision>
-          <origin
-            xyz="-2.5000000000650840986e-06 -1.1265347830754021332e-17 -4.3301270189615499146e-06"
-            rpy="-3.141592653589793116 1.0471975511965965211 3.1415926535897922278" />
-          <geometry>
-            <mesh filename="package://minipock_description/models/tire.stl" />
-          </geometry>
-        </collision>
-        <inertial>
-          <origin xyz="0 0 0" rpy="0 0 0" />
-          <mass value="0.001" />
-          <inertia ixx="0.001" ixy="0" ixz="0" iyy="0.001" iyz="0" izz="0.001" />
-        </inertial>
-        <visual>
-          <origin
-            xyz="-2.5000000000650840986e-06 -1.1265347830754021332e-17 -4.3301270189615499146e-06"
-            rpy="-3.141592653589793116 1.0471975511965965211 3.1415926535897922278" />
-          <geometry>
-            <mesh filename="package://minipock_description/models/tire.stl" />
-          </geometry>
-          <material name="${name}_rollers_11_visual_material">
-            <color
-              rgba="0.49803921568627451677 0.49803921568627451677 0.49803921568627451677 1.0" />
-          </material>
-        </visual>
-      </link>
-      <joint name="${name}_rollers_11_fixing" type="continuous">
-        <origin xyz="0 0 0" rpy="0 -0 0" />
-        <parent link="${name}_wheel_link" />
-        <child link="${name}_rollers_11" />
-        <axis xyz="0 0 1" />
-        <limit effort="1" velocity="20" />
-      </joint>
-      <link name="${name}_rollers_12">
-        <collision>
-          <origin
-            xyz="4.9999999999113253768e-06 -2.7755575615628913511e-17 6.9388939039072283776e-18"
-            rpy="1.8722173686805076642e-30 4.3675930115564019462e-15 4.8181242536834853273e-16" />
-          <geometry>
-            <mesh filename="package://minipock_description/models/tire.stl" />
-          </geometry>
-        </collision>
-        <inertial>
-          <origin xyz="0 0 0" rpy="0 0 0" />
-          <mass value="0.001" />
-          <inertia ixx="0.001" ixy="0" ixz="0" iyy="0.001" iyz="0" izz="0.001" />
-        </inertial>
-        <visual>
-          <origin
-            xyz="4.9999999999113253768e-06 -2.7755575615628913511e-17 6.9388939039072283776e-18"
-            rpy="1.8722173686805076642e-30 4.3675930115564019462e-15 4.8181242536834853273e-16" />
-          <geometry>
-            <mesh filename="package://minipock_description/models/tire.stl" />
-          </geometry>
-          <material name="${name}_rollers_12_visual_material">
-            <color
-              rgba="0.49803921568627451677 0.49803921568627451677 0.49803921568627451677 1.0" />
-          </material>
-        </visual>
-      </link>
-      <joint name="${name}_rollers_12_fixing" type="continuous">
-        <origin xyz="0 0 0" rpy="0 -0 0" />
-        <parent link="${name}_wheel_link" />
-        <child link="${name}_rollers_12" />
-        <axis xyz="0 0 1" />
-        <limit effort="1" velocity="20" />
-      </joint>
-      <link name="${name}_rollers_13">
-        <collision>
-          <origin
-            xyz="-2.5000000000402304579e-06 -2.6888213877640509963e-17 4.3301270189815763145e-06"
-            rpy="-3.1415926535897922278 -1.0471975511965989636 3.1415926535897922278" />
-          <geometry>
-            <mesh filename="package://minipock_description/models/tire.stl" />
-          </geometry>
-        </collision>
-        <inertial>
-          <origin xyz="0 0 0" rpy="0 0 0" />
-          <mass value="0.001" />
-          <inertia ixx="0.001" ixy="0" ixz="0" iyy="0.001" iyz="0" izz="0.001" />
-        </inertial>
-        <visual>
-          <origin
-            xyz="-2.5000000000402304579e-06 -2.6888213877640509963e-17 4.3301270189815763145e-06"
-            rpy="-3.1415926535897922278 -1.0471975511965989636 3.1415926535897922278" />
-          <geometry>
-            <mesh filename="package://minipock_description/models/tire.stl" />
-          </geometry>
-          <material name="${name}_rollers_13_visual_material">
-            <color
-              rgba="0.49803921568627451677 0.49803921568627451677 0.49803921568627451677 1.0" />
-          </material>
-        </visual>
-      </link>
-      <joint name="${name}_rollers_13_fixing" type="continuous">
-        <origin xyz="0 0 0" rpy="0 -0 0" />
-        <parent link="${name}_wheel_link" />
-        <child link="${name}_rollers_13" />
-        <axis xyz="0 0 1" />
-        <limit effort="1" velocity="20" />
-      </joint>
-      <link name="${name}_rollers_14">
-        <collision>
-          <origin
-            xyz="-4.9999999999078559298e-06 -2.7755575615628913511e-17 3.8163916471489756077e-17"
-            rpy="-3.141592653589793116 -4.3675930115564019462e-15 3.1415926535897926719" />
-          <geometry>
-            <mesh filename="package://minipock_description/models/tire.stl" />
-          </geometry>
-        </collision>
-        <inertial>
-          <origin xyz="0 0 0" rpy="0 0 0" />
-          <mass value="0.001" />
-          <inertia ixx="0.001" ixy="0" ixz="0" iyy="0.001" iyz="0" izz="0.001" />
-        </inertial>
-        <visual>
-          <origin
-            xyz="-4.9999999999078559298e-06 -2.7755575615628913511e-17 3.8163916471489756077e-17"
-            rpy="-3.141592653589793116 -4.3675930115564019462e-15 3.1415926535897926719" />
-          <geometry>
-            <mesh filename="package://minipock_description/models/tire.stl" />
-          </geometry>
-          <material name="${name}_rollers_14_visual_material">
-            <color
-              rgba="0.49803921568627451677 0.49803921568627451677 0.49803921568627451677 1.0" />
-          </material>
-        </visual>
-      </link>
-      <joint name="${name}_rollers_14_fixing" type="continuous">
-        <origin xyz="0 0 0" rpy="0 -0 0" />
-        <parent link="${name}_wheel_link" />
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
Commit message: refactor: Update motor.xacro to adjust wheel positions and colors

File: minipock_description/urdf/motor.xacro (robot description, xacro)
@@ -55,5 +55,5 @@
           <material name="${name}_wheel_link_material">
             <color
-              rgba="0.76862745098039220171 0.88627450980392152857 0.95294117647058818044 1.0" />
+              rgba="0.06862745098039220171 0.08627450980392152857 0.05294117647058818044 1.0" />
           </material>
         </visual>
@@ -71,5 +71,5 @@
         <parent link="${name}_base_link" />
         <child link="${name}_wheel_link" />
-        <origin xyz="0.0 0.05 0.024" rpy="${pi/2} 0 0" />
+        <origin xyz="0.0 0.02 0.024" rpy="${pi/2} 0 0" />
         <axis xyz="0 0 ${side}" />
         <limit effort="2000" velocity="45.5" />
@@ -84,5 +84,5 @@
           <material name="roller_material">
             <color
-              rgba="0.64705882352941179736 0.64705882352941179736 0.64705882352941179736 1.0" />
+              rgba="0.14705882352941179736 0.14705882352941179736 0.14705882352941179736 1.0" />
           </material>
         </visual>
@@ -121,5 +121,5 @@
           <material name="roller_material">
             <color
-              rgba="0.64705882352941179736 0.64705882352941179736 0.64705882352941179736 1.0" />
+              rgba="0.14705882352941179736 0.14705882352941179736 0.14705882352941179736 1.0" />
           </material>
         </visual>
@@ -158,5 +158,5 @@
           <material name="roller_material">
             <color
-              rgba="0.64705882352941179736 0.64705882352941179736 0.64705882352941179736 1.0" />
+              rgba="0.14705882352941179736 0.14705882352941179736 0.14705882352941179736 1.0" />
           </material>
         </visual>
@@ -195,5 +195,5 @@
           <material name="roller_material">
             <color
-              rgba="0.64705882352941179736 0.64705882352941179736 0.64705882352941179736 1.0" />
+              rgba="0.14705882352941179736 0.14705882352941179736 0.14705882352941179736 1.0" />
           </material>
         </visual>
@@ -232,5 +232,5 @@
           <material name="roller_material">
             <color
-              rgba="0.64705882352941179736 0.64705882352941179736 0.64705882352941179736 1.0" />
+              rgba="0.14705882352941179736 0.14705882352941179736 0.14705882352941179736 1.0" />
           </material>
         </visual>
@@ -269,5 +269,5 @@
           <material name="roller_material">
             <color
-              rgba="0.64705882352941179736 0.64705882352941179736 0.64705882352941179736 1.0" />
+              rgba="0.14705882352941179736 0.14705882352941179736 0.14705882352941179736 1.0" />
           </material>
         </visual>
@@ -307,5 +307,5 @@
           <material name="roller_material">
             <color
-              rgba="0.64705882352941179736 0.64705882352941179736 0.64705882352941179736 1.0" />
+              rgba="0.14705882352941179736 0.14705882352941179736 0.14705882352941179736 1.0" />
           </material>
         </visual>
@@ -345,5 +345,5 @@
           <material name="roller_material">
             <color
-              rgba="0.64705882352941179736 0.64705882352941179736 0.64705882352941179736 1.0" />
+              rgba="0.14705882352941179736 0.14705882352941179736 0.14705882352941179736 1.0" />
           </material>
         </visual>
@@ -372,4 +372,42 @@
         <axis xyz="0 0 1" />
         <limit effort="1" velocity="20" />
+      </joint>
+      <link name="${name}_roller_9">
+        <visual>
+          <origin xyz="0 0 -0.0080000000000000001665"
+            rpy="6.7221822527689735584e-18 -8.7180519648836596984e-33 -1.2569312029751666415e-31" />
+          <geometry>
+            <mesh filename="package://minipock_description/models/roller.stl" />
+          </geometry>
+          <material name="roller_material">
+            <color
+              rgba="0.14705882352941179736 0.14705882352941179736 0.14705882352941179736 1.0" />
+          </material>
+        </visual>
+        <collision>
+          <origin xyz="0 0 -0.0080000000000000001665"
+            rpy="6.7221822527689735584e-18 -8.7180519648836596984e-33 -1.2569312029751666415e-31" />
+          <geometry>
+            <mesh filename="package://minipock_description/models/roller.stl" />
+          </geometry>
+        </collision>
+        <inertial>
+          <origin
+            xyz="4.0653990009220675453e-20 2.3540384680750280962e-32 -0.0079999999999998284289"
+            rpy="0 0 0" />
+          <mass value="0.0015147722925255755443" />
+          <inertia ixx="4.0501606036357593342e-08" ixy="-4.6621608404600178297e-39"
+            ixz="-6.5460416771372355481e-39" iyy="4.0501606036357593342e-08"
+            iyz="4.055471787642257058e-24" izz="2.7582542641814991776e-08" />
+        </inertial>
+      </link>
+      <joint name="${name}_joint_roller_7_continuous" type="continuous">
+        <origin xyz="-0.013258688745465072728 0.028036857843754141306 -0.0049999999999999992367"
+          rpy="-0.69813170079771968979 1.5707963267948958919 0" />
+        <parent link="${name}_wheel_link" />
+        <child link="${name}_roller_9" />
+        <axis xyz="0 0 1" />
+        <limit effort="1" velocity="20" />
+        <joint_properties friction="0.0" />
       </joint>
     </xacro:if>
