Commit message: refactor: Update motor.xacro to increase wheel velocity limits

File: minipock_description/urdf/motor.xacro (robot description, xacro)
@@ -110,5 +110,5 @@
         <child link="${name}_roller" />
         <axis xyz="0 0 1" />
-        <limit effort="1" velocity="20" />
+         <limit effort="1" velocity="200" />
       </joint>
       <link name="${name}_roller_2">
@@ -147,5 +147,5 @@
         <child link="${name}_roller_2" />
         <axis xyz="0 0 1" />
-        <limit effort="1" velocity="20" />
+         <limit effort="1" velocity="200" />
       </joint>
       <link name="${name}_roller_3">
@@ -184,5 +184,5 @@
         <child link="${name}_roller_3" />
         <axis xyz="0 0 1" />
-        <limit effort="1" velocity="20" />
+         <limit effort="1" velocity="200" />
       </joint>
       <link name="${name}_roller_4">
@@ -221,5 +221,5 @@
         <child link="${name}_roller_4" />
         <axis xyz="0 0 1" />
-        <limit effort="1" velocity="20" />
+         <limit effort="1" velocity="200" />
       </joint>
       <link name="${name}_roller_5">
@@ -258,5 +258,5 @@
         <child link="${name}_roller_5" />
         <axis xyz="0 0 1" />
-        <limit effort="1" velocity="20" />
+         <limit effort="1" velocity="200" />
       </joint>
       <link name="${name}_roller_6">
@@ -295,5 +295,5 @@
         <child link="${name}_roller_6" />
         <axis xyz="0 0 1" />
-        <limit effort="1" velocity="20" />
+         <limit effort="1" velocity="200" />
       </joint>
       <link name="${name}_roller_7">
@@ -334,5 +334,5 @@
         <child link="${name}_roller_7" />
         <axis xyz="0 0 1" />
-        <limit effort="1" velocity="20" />
+         <limit effort="1" velocity="200" />
       </joint>
       <link name="${name}_roller_8">
@@ -371,5 +371,5 @@
         <child link="${name}_roller_8" />
         <axis xyz="0 0 1" />
-        <limit effort="1" velocity="20" />
+         <limit effort="1" velocity="200" />
       </joint>
       <link name="${name}_roller_9">
@@ -408,5 +408,5 @@
         <child link="${name}_roller_9" />
         <axis xyz="0 0 1" />
-        <limit effort="1" velocity="20" />
+         <limit effort="1" velocity="200" />
         <joint_properties friction="0.0" />
       </joint>
@@ -421,5 +421,5 @@
         name="gz::sim::systems::JointController">
         <joint_name>${name}_wheel_joint</joint_name>
-        <use_velocity_commands>true</use_velocity_commands>
+        <use_velocity_commands>false</use_velocity_commands>
         <topic>${namespace}${name}/pos</topic>
         <name>${name}</name>
