Commit message: Update sensors.xacro and spawn.launch.py for minipock_gz package

File: minipock_description/urdf/sensors.xacro (robot description, xacro)
@@ -5,5 +5,5 @@
     <link name="${namespace}${name}_link">
       <visual name="${name}_visual">
-        <origin xyz="0 0 0" rpy="${pi/2} 0 0"/>
+        <origin xyz="0 0 0" rpy="${pi/2} ${pi} 0"/>
         <geometry>
           <mesh filename="package://minipock_description/models/lds_visual.dae"/>
