Commit message: refactor: Update minipock_base.xacro to use cylinder geometry for the collision

File: minipock_description/urdf/minipock_base.xacro (robot description, xacro)
@@ -12,5 +12,5 @@
         <origin xyz="0 0 -${0.089/2}" rpy="0 -0 ${-pi/2}" />
         <geometry>
-          <box size="0.30 0.342 0.089" />
+          <cylinder radius="0.15" length="0.089" />
         </geometry>
       </collision>

Commit message: Update minipock_description/urdf/minipock_base.xacro and minipock_description/urdf/sensors.xacro

File: minipock_description/urdf/minipock_base.xacro (robot description, xacro)
@@ -14,10 +14,10 @@
         <origin xyz="0 0 -${0.089/2}" rpy="0 -0 ${-pi/2}" />
         <geometry>
-          <cylinder radius="0.15" length="0.089" />
+          <cylinder radius="0.15" length="0.092" />
         </geometry>
       </collision>
       <inertial>
         <origin xyz="0.0 -0.029 0.0" rpy="0 -0 0" />
-        <mass value="1.587" />
+        <mass value="7.587" />
         <inertia ixx="0.014" ixy="0.0" ixz="0.0" iyy="0.025" iyz="0.0" izz="0.013" />
       </inertial>

File: minipock_description/urdf/sensors.xacro (robot description, xacro)
@@ -30,5 +30,5 @@
     <gazebo reference="${namespace}${name}_link">
       <sensor type="gpu_lidar" name="lds_01">
-        <update_rate>50</update_rate>
+        <update_rate>10</update_rate>
         <topic>${namespace}scan_raw</topic>
         <visualize>true</visualize>
@@ -43,6 +43,6 @@
           </scan>
           <range>
-            <min>0.12</min>
-            <max>3.5</max>
+            <min>0.5</min>
+            <max>12.0</max>
             <resolution>0.0150</resolution>
           </range>
