Commit message: fix : change base_link to ${namespace}base_link and set as blank

File: minipock_description/urdf/minipock.urdf.xacro (robot description, xacro)
@@ -1,19 +1,23 @@
 <?xml version="1.0"?>
 <robot name="minipock" xmlns:xacro="http://ros.org/wiki/xacro">
-  <xacro:property name="namespace" value="minipock"/>
-  <xacro:include filename="$(find minipock_description)/urdf/minipock_differential_base.xacro"/>
-  <xacro:minipock_base namespace="${namespace}"/>
+  <xacro:property name="namespace" value="" />
+  <xacro:include filename="$(find minipock_description)/urdf/minipock_differential_base.xacro" />
+  <xacro:minipock_base namespace="${namespace}" name="minipock" />
   <!-- motor -->
-  <xacro:include filename="$(find minipock_description)/urdf/motor_stepper.xacro"/>
-  <xacro:motor_stepper namespace="${namespace}" name="stepper_left" x="0.0" y="0.133" z="-0.086" R="0.0" P="0.0"
-                       Y="0.0" side="1"/>
-  <xacro:motor_stepper namespace="${namespace}" name="stepper_right" x="0.0" y="-0.133" z="-0.086" R="0.0" P="0.0"
-                       Y="${-pi}" side="-1"/>
-  <xacro:include filename="$(find minipock_description)/urdf/sensors.xacro"/>
-  <xacro:lds_01 namespace="${namespace}" name="lds_01" x="0.0" y="0.0" z="0.050" R="0.0" P="0.0" Y="${pi}"/>
+  <xacro:include filename="$(find minipock_description)/urdf/motor_stepper.xacro" />
+  <xacro:motor_stepper namespace="${namespace}" name="stepper_left" x="0.0" y="0.133" z="-0.086"
+    R="0.0" P="0.0"
+    Y="0.0" side="1" />
+  <xacro:motor_stepper namespace="${namespace}" name="stepper_right" x="0.0" y="-0.133" z="-0.086"
+    R="0.0" P="0.0"
+    Y="${-pi}" side="-1" />
+  <!-- sensors -->
+  <xacro:include filename="$(find minipock_description)/urdf/sensors.xacro" />
+  <xacro:lds_01 namespace="${namespace}" name="lds_01" x="0.0" y="0.0" z="0.050" R="0.0" P="0.0"
+    Y="${pi}" />
   <gazebo>
     <plugin
-        filename="gz-sim-diff-drive-system"
-        name="gz::sim::systems::DiffDrive">
+      filename="gz-sim-diff-drive-system"
+      name="gz::sim::systems::DiffDrive">
       <left_joint>stepper_left_wheel_joint</left_joint>
       <right_joint>stepper_right_wheel_joint</right_joint>
@@ -22,9 +26,9 @@
       <odom_publish_frequency>50</odom_publish_frequency>
       <topic>cmd_vel</topic>
-      <child_frame_id>base_link</child_frame_id>
+      <child_frame_id>${namespace}base_link</child_frame_id>
       <frame_id>odom</frame_id>
     </plugin>
     <plugin filename="libgz-sim-pose-publisher-system.so"
-            name="gz::sim::systems::PosePublisher">
+      name="gz::sim::systems::PosePublisher">
       <publish_link_pose>false</publish_link_pose>
       <publish_sensor_pose>true</publish_sensor_pose>
@@ -38,6 +42,6 @@
     </plugin>
     <plugin
-        filename="gz-sim-joint-state-publisher-system"
-        name="gz::sim::systems::JointStatePublisher">
+      filename="gz-sim-joint-state-publisher-system"
+      name="gz::sim::systems::JointStatePublisher">
     </plugin>
   </gazebo>

File: minipock_description/urdf/minipock_differential_base.xacro (robot description, xacro)
@@ -1,71 +1,71 @@
 <?xml version="1.0"?>
 <robot name="minipock" xmlns:xacro="http://ros.org/wiki/xacro">
-  <xacro:macro name="minipock_base" params="namespace:=minipock">
-    <link name="base_link">
+  <xacro:macro name="minipock_base" params="namespace:=minipock name:=minipock">
+    <link name="${namespace}base_link">
       <visual>
-        <origin xyz="0 0 0.0" rpy="0 0 ${-pi/2}"/>
+        <origin xyz="0 0 0.0" rpy="0 0 ${-pi/2}" />
         <geometry>
-          <mesh filename="package://minipock_description/models/differential_base_alu.dae"/>
+          <mesh filename="package://minipock_description/models/differential_base_alu.dae" />
         </geometry>
       </visual>
       <collision>
-        <origin xyz="0 0 -${0.089/2}" rpy="0 -0 ${-pi/2}"/>
+        <origin xyz="0 0 -${0.089/2}" rpy="0 -0 ${-pi/2}" />
         <geometry>
-          <box size="0.30 0.342 0.089"/>
+          <box size="0.30 0.342 0.089" />
         </geometry>
       </collision>
       <inertial>
-        <origin xyz="0.0 -0.029 0.0" rpy="0 -0 0"/>
-        <mass value="1.587"/>
-        <inertia ixx="0.014" ixy="0.0" ixz="0.0" iyy="0.025" iyz="0.0" izz="0.013"/>
+        <origin xyz="0.0 -0.029 0.0" rpy="0 -0 0" />
+        <mass value="1.587" />
+        <inertia ixx="0.014" ixy="0.0" ixz="0.0" iyy="0.025" iyz="0.0" izz="0.013" />
       </inertial>
     </link>
-    <link name="${namespace}_structure_pla_link">
+    <link name="${name}_structure_pla_link">
       <visual>
-        <origin xyz="0 0 0.0" rpy="0 0 0"/>
+        <origin xyz="0 0 0.0" rpy="0 0 0" />
         <geometry>
-          <mesh filename="package://minipock_description/models/differential_base_pla.stl"/>
+          <mesh filename="package://minipock_description/models/differential_base_pla.stl" />
         </geometry>
         <material name="6TRON">
-          <color rgba="0.27 0.64 0.52 1.0"/>
+          <color rgba="0.27 0.64 0.52 1.0" />
         </material>
       </visual>
     </link>
-    <link name="${namespace}_structure_pmma_link">
+    <link name="${name}_structure_pmma_link">
       <visual>
-        <origin xyz="0 0 0.0" rpy="0 0 0"/>
+        <origin xyz="0 0 0.0" rpy="0 0 0" />
         <geometry>
-          <mesh filename="package://minipock_description/models/differential_base_pmma.stl"/>
+          <mesh filename="package://minipock_description/models/differential_base_pmma.stl" />
         </geometry>
         <material name="6TRON_2">
-          <color rgba="0.27 0.64 0.52 0.9"/>
+          <color rgba="0.27 0.64 0.52 0.9" />
         </material>
       </visual>
     </link>
-    <link name="${namespace}_structure_misc_link">
+    <link name="${name}_structure_misc_link">
       <visual>
-        <origin xyz="0 0 0.0" rpy="0 0 0"/>
+        <origin xyz="0 0 0.0" rpy="0 0 0" />
         <geometry>
-          <mesh filename="package://minipock_description/models/differential_misc.stl"/>
+          <mesh filename="package://minipock_description/models/differential_misc.stl" />
         </geometry>
         <material name="6TRON_2">
-          <color rgba="0.27 0.64 0.52 1.0"/>
-      </material>
+          <color rgba="0.27 0.64 0.52 1.0" />
+        </material>
       </visual>
     </link>
-    <joint name="${namespace}_structure_pla_joint" type="fixed">
-      <origin xyz="0 0 0.0" rpy="0 0 ${-pi/2}"/>
-      <parent link="base_link"/>
-      <child link="${namespace}_structure_pla_link"/>
+    <joint name="${name}_structure_pla_joint" type="fixed">
+      <origin xyz="0 0 0.0" rpy="0 0 ${-pi/2}" />
+      <parent link="${namespace}base_link" />
+      <child link="${name}_structure_pla_link" />
     </joint>
-    <joint name="${namespace}_structure_pmma_joint" type="fixed">
-      <origin xyz="0 0 0.0" rpy="0 0 ${-pi/2}"/>
-      <parent link="base_link"/>
-      <child link="${namespace}_structure_pmma_link"/>
+    <joint name="${name}_structure_pmma_joint" type="fixed">
+      <origin xyz="0 0 0.0" rpy="0 0 ${-pi/2}" />
+      <parent link="${namespace}base_link" />
+      <child link="${name}_structure_pmma_link" />
     </joint>
-    <joint name="${namespace}_structure_misc_joint" type="fixed">
-      <origin xyz="0 0 0.0" rpy="0 0 ${-pi/2}"/>
-      <parent link="base_link"/>
-      <child link="${namespace}_structure_misc_link"/>
+    <joint name="${name}_structure_misc_joint" type="fixed">
+      <origin xyz="0 0 0.0" rpy="0 0 ${-pi/2}" />
+      <parent link="${namespace}base_link" />
+      <child link="${name}_structure_misc_link" />
     </joint>
   </xacro:macro>

File: minipock_description/urdf/motor_stepper.xacro (robot description, xacro)
@@ -37,5 +37,5 @@
     </link>
     <joint name="${name}_joint" type="fixed">
-      <parent link="base_link" />
+      <parent link="${namespace}base_link" />
       <child link="${name}_base_link" />
       <origin xyz="${x} ${y} ${z}" rpy="${R} ${P} ${Y}" />
@@ -54,5 +54,5 @@
         <joint_name>${name}_wheel_joint</joint_name>
         <use_velocity_commands>true</use_velocity_commands>
-        <topic>${namespace}/${name}/pos</topic>
+        <topic>${namespace}${name}/pos</topic>
         <name>${name}</name>
       </plugin>

File: minipock_description/urdf/sensors.xacro (robot description, xacro)
@@ -24,5 +24,5 @@
       <limit effort="1000.0" lower="0.0" upper="0" velocity="0"/>
       <origin xyz="${x} ${y} ${z}" rpy="${R} ${P} ${Y}"/>
-      <parent link="base_link"/>
+      <parent link="${namespace}base_link"/>
       <child link="${name}_link"/>
     </joint>

Commit message: feat: Update minipock_description to use new base model filenames

File: minipock_description/urdf/minipock.urdf.xacro (robot description, xacro)
@@ -2,5 +2,5 @@
 <robot name="minipock" xmlns:xacro="http://ros.org/wiki/xacro">
   <xacro:property name="namespace" value="" />
-  <xacro:include filename="$(find minipock_description)/urdf/minipock_differential_base.xacro" />
+  <xacro:include filename="$(find minipock_description)/urdf/minipock_base.xacro" />
   <xacro:minipock_base namespace="${namespace}" name="minipock" />
   <!-- motor -->

File: minipock_description/urdf/minipock_base.xacro (robot description, xacro)
@@ -6,5 +6,5 @@
         <origin xyz="0 0 0.0" rpy="0 0 ${-pi/2}" />
         <geometry>
-          <mesh filename="package://minipock_description/models/differential_base_alu.dae" />
+          <mesh filename="package://minipock_description/models/base_alu.dae" />
         </geometry>
       </visual>
@@ -25,5 +25,5 @@
         <origin xyz="0 0 0.0" rpy="0 0 0" />
         <geometry>
-          <mesh filename="package://minipock_description/models/differential_base_pla.stl" />
+          <mesh filename="package://minipock_description/models/base_pla.stl" />
         </geometry>
         <material name="6TRON">
@@ -36,5 +36,5 @@
         <origin xyz="0 0 0.0" rpy="0 0 0" />
         <geometry>
-          <mesh filename="package://minipock_description/models/differential_base_pmma.stl" />
+          <mesh filename="package://minipock_description/models/base_pmma.stl" />
         </geometry>
         <material name="6TRON_2">
@@ -47,5 +47,5 @@
         <origin xyz="0 0 0.0" rpy="0 0 0" />
         <geometry>
-          <mesh filename="package://minipock_description/models/differential_misc.stl" />
+          <mesh filename="package://minipock_description/models/misc.stl" />
         </geometry>
         <material name="6TRON_2">

Commit message: feat: use differential mode for motor_stepper if mode is set to 'differential'

File: minipock_description/urdf/minipock.urdf.xacro (robot description, xacro)
@@ -2,14 +2,17 @@
 <robot name="minipock" xmlns:xacro="http://ros.org/wiki/xacro">
   <xacro:property name="namespace" value="" />
+  <xacro:property name="mode" value="differential" />
   <xacro:include filename="$(find minipock_description)/urdf/minipock_base.xacro" />
   <xacro:minipock_base namespace="${namespace}" name="minipock" />
   <!-- motor -->
   <xacro:include filename="$(find minipock_description)/urdf/motor_stepper.xacro" />
-  <xacro:motor_stepper namespace="${namespace}" name="stepper_left" x="0.0" y="0.133" z="-0.086"
-    R="0.0" P="0.0"
-    Y="0.0" side="1" />
-  <xacro:motor_stepper namespace="${namespace}" name="stepper_right" x="0.0" y="-0.133" z="-0.086"
-    R="0.0" P="0.0"
-    Y="${-pi}" side="-1" />
+  <xacro:if value="${mode == 'differential'}">
+    <xacro:motor_stepper namespace="${namespace}" name="stepper_left" x="0.0" y="0.133" z="-0.086"
+      R="0.0" P="0.0"
+      Y="0.0" side="1" />
+    <xacro:motor_stepper namespace="${namespace}" name="stepper_right" x="0.0" y="-0.133" z="-0.086"
+      R="0.0" P="0.0"
+      Y="${-pi}" side="-1" />
+  </xacro:if>
   <!-- sensors -->
   <xacro:include filename="$(find minipock_description)/urdf/sensors.xacro" />
@@ -17,16 +20,18 @@
     Y="${pi}" />
   <gazebo>
-    <plugin
-      filename="gz-sim-diff-drive-system"
-      name="gz::sim::systems::DiffDrive">
-      <left_joint>stepper_left_wheel_joint</left_joint>
-      <right_joint>stepper_right_wheel_joint</right_joint>
-      <wheel_separation>0.335</wheel_separation>
-      <wheel_radius>0.036</wheel_radius>
-      <odom_publish_frequency>50</odom_publish_frequency>
-      <topic>cmd_vel</topic>
-      <child_frame_id>${namespace}base_link</child_frame_id>
-      <frame_id>odom</frame_id>
-    </plugin>
+    <xacro:if value="${mode == 'differential'}">
+      <plugin
+        filename="gz-sim-diff-drive-system"
+        name="gz::sim::systems::DiffDrive">
+        <left_joint>stepper_left_wheel_joint</left_joint>
+        <right_joint>stepper_right_wheel_joint</right_joint>
+        <wheel_separation>0.335</wheel_separation>
+        <wheel_radius>0.036</wheel_radius>
+        <odom_publish_frequency>50</odom_publish_frequency>
+        <topic>cmd_vel</topic>
+        <child_frame_id>${namespace}base_link</child_frame_id>
+        <frame_id>odom</frame_id>
+      </plugin>
+    </xacro:if>
     <plugin filename="libgz-sim-pose-publisher-system.so"
       name="gz::sim::systems::PosePublisher">

Commit message: refactor: change stepper to motor in minipock_description

File: minipock_description/urdf/minipock.urdf.xacro (robot description, xacro)
@@ -6,12 +6,23 @@
   <xacro:minipock_base namespace="${namespace}" name="minipock" />
   <!-- motor -->
-  <xacro:include filename="$(find minipock_description)/urdf/motor_stepper.xacro" />
+  <xacro:include filename="$(find minipock_description)/urdf/motor.xacro" />
   <xacro:if value="${mode == 'differential'}">
-    <xacro:motor_stepper namespace="${namespace}" name="stepper_left" x="0.0" y="0.133" z="-0.086"
+    <xacro:motor namespace="${namespace}" name="motor_left" x="0.0" y="0.133" z="-0.086"
       R="0.0" P="0.0"
       Y="0.0" side="1" />
-    <xacro:motor_stepper namespace="${namespace}" name="stepper_right" x="0.0" y="-0.133" z="-0.086"
+    <xacro:motor namespace="${namespace}" name="motor_right" x="0.0" y="-0.133" z="-0.086"
       R="0.0" P="0.0"
       Y="${-pi}" side="-1" />
+  </xacro:if>
+  <xacro:if value="${mode == 'holonomic'}">
+    <xacro:motor namespace="${namespace}" name="motor_left" x="0.0" y="0.133" z="-0.086"
+      R="0.0" P="0.0"
+      Y="0.0" side="1" />
+    <xacro:motor namespace="${namespace}" name="motor_right" x="0.0" y="-0.133" z="-0.086"
+      R="0.0" P="0.0"
+      Y="${-pi}" side="-1" />
+    <xacro:motor namespace="${namespace}" name="motor_middle" x="0.150" y="0.0" z="-0.086"
+      R="0.0" P="0.0"
+      Y="${-pi/2}" side="-1" />
   </xacro:if>
   <!-- sensors -->
@@ -24,6 +35,6 @@
         filename="gz-sim-diff-drive-system"
         name="gz::sim::systems::DiffDrive">
-        <left_joint>stepper_left_wheel_joint</left_joint>
-        <right_joint>stepper_right_wheel_joint</right_joint>
+        <left_joint>motor_left_wheel_joint</left_joint>
+        <right_joint>motor_right_wheel_joint</right_joint>
         <wheel_separation>0.335</wheel_separation>
         <wheel_radius>0.036</wheel_radius>

File: minipock_description/urdf/motor.xacro (robot description, xacro)
@@ -1,6 +1,6 @@
 <?xml version="1.0"?>
 <robot name="minipock" xmlns:xacro="http://ros.org/wiki/xacro">
-  <xacro:macro name="motor_stepper"
-    params="namespace:=minipock name:=stepper_left x:=0.0 y:=0.0 z:=0.0
+  <xacro:macro name="motor"
+    params="namespace:=minipock name:=motor_left x:=0.0 y:=0.0 z:=0.0
 				       R:=0.0 P:=0.0 Y:=0.0 side:=1">
     <link name="${name}_base_link">

Commit message: feat: use holonomic mode for motor and motor_stepper

File: minipock_description/urdf/minipock.urdf.xacro (robot description, xacro)
@@ -2,5 +2,5 @@
 <robot name="minipock" xmlns:xacro="http://ros.org/wiki/xacro">
   <xacro:property name="namespace" value="" />
-  <xacro:property name="mode" value="differential" />
+  <xacro:property name="mode" value="holonomic" />
   <xacro:include filename="$(find minipock_description)/urdf/minipock_base.xacro" />
   <xacro:minipock_base namespace="${namespace}" name="minipock" />
@@ -16,13 +16,13 @@
   </xacro:if>
   <xacro:if value="${mode == 'holonomic'}">
-    <xacro:motor namespace="${namespace}" name="motor_left" x="0.0" y="0.133" z="-0.086"
+    <xacro:motor namespace="${namespace}" name="motor_left" x="0.0" y="0.145" z="-0.086"
       R="0.0" P="0.0"
       Y="0.0" side="1" />
-    <xacro:motor namespace="${namespace}" name="motor_right" x="0.0" y="-0.133" z="-0.086"
+    <xacro:motor namespace="${namespace}" name="motor_right" x="-0.126" y="-0.073" z="-0.086"
       R="0.0" P="0.0"
-      Y="${-pi}" side="-1" />
-    <xacro:motor namespace="${namespace}" name="motor_middle" x="0.150" y="0.0" z="-0.086"
+      Y="${120*pi/180}" side="1" />
+    <xacro:motor namespace="${namespace}" name="motor_middle" x="0.126" y="-0.073" z="-0.086"
       R="0.0" P="0.0"
-      Y="${-pi/2}" side="-1" />
+      Y="${240*pi/180}" side="1" />
   </xacro:if>
   <!-- sensors -->

Commit message: feat: change motor max velocity

File: minipock_description/urdf/minipock.urdf.xacro (robot description, xacro)
@@ -2,5 +2,5 @@
 <robot name="minipock" xmlns:xacro="http://ros.org/wiki/xacro">
   <xacro:property name="namespace" value="" />
-  <xacro:property name="mode" value="holonomic" />
+  <xacro:property name="mode" value="differential" />
   <xacro:include filename="$(find minipock_description)/urdf/minipock_base.xacro" />
   <xacro:minipock_base namespace="${namespace}" name="minipock" />

File: minipock_description/urdf/motor.xacro (robot description, xacro)
@@ -46,5 +46,5 @@
       <origin xyz="0.0 0.0 0.024" rpy="0 0 0" />
       <axis xyz="0 ${side} 0" />
-      <limit effort="2000" velocity="5" />
+      <limit effort="2000" velocity="45.5"/>
     </joint>
     <gazebo>
