Commit message: feat: add holonomic option for wheel
updates the `minipock_description` package by modifying the `motos.xacro` to add holonomic wheel

File: minipock_description/urdf/minipock.urdf.xacro (robot description, xacro)
@@ -9,20 +9,15 @@
   <xacro:if value="${mode == 'differential'}">
     <xacro:motor namespace="${namespace}" name="motor_left" x="0.0" y="0.133" z="-0.086"
-      R="0.0" P="0.0"
-      Y="0.0" side="1" />
+      R="0.0" P="0.0" Y="0.0" side="1" mode="${mode}" />
     <xacro:motor namespace="${namespace}" name="motor_right" x="0.0" y="-0.133" z="-0.086"
-      R="0.0" P="0.0"
-      Y="${-pi}" side="-1" />
+      R="0.0" P="0.0" Y="${-pi}" side="-1" mode="${mode}" />
   </xacro:if>
   <xacro:if value="${mode == 'holonomic'}">
     <xacro:motor namespace="${namespace}" name="motor_left" x="0.0" y="0.145" z="-0.086"
-      R="0.0" P="0.0"
-      Y="0.0" side="1" />
+      R="0.0" P="0.0" Y="0.0" side="1" mode="${mode}"/>
     <xacro:motor namespace="${namespace}" name="motor_right" x="-0.126" y="-0.073" z="-0.086"
-      R="0.0" P="0.0"
-      Y="${120*pi/180}" side="1" />
+      R="0.0" P="0.0" Y="${120*pi/180}" side="1" mode="${mode}"/>
     <xacro:motor namespace="${namespace}" name="motor_middle" x="0.126" y="-0.073" z="-0.086"
-      R="0.0" P="0.0"
-      Y="${240*pi/180}" side="1" />
+      R="0.0" P="0.0" Y="${240*pi/180}" side="1" mode="${mode}"/>
   </xacro:if>
   <!-- sensors -->

File: minipock_description/urdf/motor.xacro (robot description, xacro)
@@ -3,5 +3,5 @@
   <xacro:macro name="motor"
     params="namespace:=minipock name:=motor_left x:=0.0 y:=0.0 z:=0.0
-				       R:=0.0 P:=0.0 Y:=0.0 side:=1">
+				       R:=0.0 P:=0.0 Y:=0.0 side:=1 mode:='differential'">
     <link name="${name}_base_link">
       <visual>
@@ -17,34 +17,99 @@
       </inertial>
     </link>
-    <link name="${name}_wheel_link">
-      <visual>
-        <origin xyz="0 0 -0.024" rpy="${pi/2} 0 0" />
-        <geometry>
-          <mesh filename="package://minipock_description/models/wheel_rotative.dae" />
-        </geometry>
-      </visual>
-      <collision>
-        <origin xyz="0 0.032 0.0" rpy="${pi/2} -0 0" />
-        <geometry>
-          <cylinder radius="0.036" length="0.006" />
-        </geometry>
-      </collision>
-      <inertial>
-        <origin xyz="0.0 -0.029 0.0" rpy="0 -0 0" />
-        <mass value="1.587" />
-        <inertia ixx="0.014" ixy="0.0" ixz="0.0" iyy="0.025" iyz="0.0" izz="0.013" />
-      </inertial>
-    </link>
+    <xacro:if value="${mode == 'differential'}">
+      <link name="${name}_wheel_link">
+        <visual>
+          <origin xyz="0 0 -0.024" rpy="${pi/2} 0 0" />
+          <geometry>
+            <mesh filename="package://minipock_description/models/wheel_rotative.dae" />
+          </geometry>
+        </visual>
+        <collision>
+          <origin xyz="0 0.032 0.0" rpy="${pi/2} -0 0" />
+          <geometry>
+            <cylinder radius="0.036" length="0.006" />
+          </geometry>
+        </collision>
+        <inertial>
+          <origin xyz="0.0 -0.029 0.0" rpy="0 -0 0" />
+          <mass value="1.587" />
+          <inertia ixx="0.014" ixy="0.0" ixz="0.0" iyy="0.025" iyz="0.0" izz="0.013" />
+        </inertial>
+      </link>
+      <joint name="${name}_wheel_joint" type="continuous">
+        <parent link="${name}_base_link" />
+        <child link="${name}_wheel_link" />
+        <origin xyz="0.0 0.0 0.024" rpy="0 0 0" />
+        <axis xyz="0 ${side} 0" />
+        <limit effort="2000" velocity="45.5" />
+      </joint>
+    </xacro:if>
+    <xacro:if value="${mode == 'holonomic'}">
+      <link name="${name}_wheel_link">
+        <visual>
+          <origin xyz="0 0 0" rpy="0 -0 0" />
+          <geometry>
+            <mesh filename="package://minipock_description/models/core.stl" />
+          </geometry>
+          <material name="core_material">
+            <color
+              rgba="0.91764705882352937127 0.91764705882352937127 0.91764705882352937127 1.0" />
+          </material>
+        </visual>
+        <collision>
+          <origin xyz="0 0 0" rpy="0 -0 0" />
+          <geometry>
+            <mesh filename="package://minipock_description/models/side.stl" />
+          </geometry>
+        </collision>
+        <inertial>
+          <origin xyz="0.0 -0.029 0.0" rpy="0 -0 0" />
+          <mass value="1.587" />
+          <inertia ixx="0.014" ixy="0.0" ixz="0.0" iyy="0.025" iyz="0.0" izz="0.013" />
+        </inertial>
+      </link>
+      <link name="${name}_rollers">
+        <visual>
+          <origin
+            xyz="0.00449999999999999966 -0.019500000000000017319 0.0071250000000000722478"
+            rpy="-3.141592653589793116 -0.52359877559829481886 1.570796326794896558" />
+          <geometry>
+            <mesh filename="package://minipock_description/models/tire.stl" />
+          </geometry>
+        </visual>
+        <collision>
+          <origin
+            xyz="0.00449999999999999966 -0.019500000000000017319 0.0071250000000000722478"
+            rpy="-3.141592653589793116 -0.52359877559829481886 1.570796326794896558" />
+          <geometry>
+            <mesh filename="package://minipock_description/models/tire.stl" />
+          </geometry>
+        </collision>
+        <inertial>
+          <origin xyz="0.0 -0.029 0.0" rpy="0 -0 0" />
+          <mass value="1.587" />
+          <inertia ixx="0.014" ixy="0.0" ixz="0.0" iyy="0.025" iyz="0.0" izz="0.013" />
+        </inertial>
+      </link>
+      <joint name="${name}_wheel_joint" type="continuous">
+        <parent link="${name}_base_link" />
+        <child link="${name}_wheel_link" />
+        <origin xyz="0.0 0.05 0.024" rpy="0 0 0" />
+        <axis xyz="0 ${side} 0" />
+        <limit effort="2000" velocity="45.5" />
+      </joint>
+      <joint name="${name}_continuous_roller_11" type="continuous">
+        <origin xyz="-0.0071249999999999967873 -0.00449999999999999966 0.019500000000000045075"
+          rpy="1.5707963267949005548 -0 1.570796326794896558" />
+        <parent link="${name}_wheel_link" />
+        <child link="${name}_rollers" />
+        <axis xyz="0 0 1" />
+        <limit effort="1" velocity="20" />
+      </joint>
+    </xacro:if>
     <joint name="${name}_joint" type="fixed">
       <parent link="${namespace}base_link" />
       <child link="${name}_base_link" />
       <origin xyz="${x} ${y} ${z}" rpy="${R} ${P} ${Y}" />
-    </joint>
-    <joint name="${name}_wheel_joint" type="continuous">
-      <parent link="${name}_base_link" />
-      <child link="${name}_wheel_link" />
-      <origin xyz="0.0 0.0 0.024" rpy="0 0 0" />
-      <axis xyz="0 ${side} 0" />
-      <limit effort="2000" velocity="45.5"/>
     </joint>
     <gazebo>

Commit message: feat: Add namespace and update link names in minipock description

File: minipock_description/urdf/minipock.urdf.xacro (robot description, xacro)
@@ -1,8 +1,15 @@
 <?xml version="1.0"?>
 <robot name="minipock" xmlns:xacro="http://ros.org/wiki/xacro">
-  <xacro:property name="namespace" value="" />
+  <xacro:arg name="namespace" default="minipock/"/>
+  <xacro:arg name="x" default="0.0"/>
+  <xacro:arg name="y" default="0.0"/>
+  <xacro:arg name="z" default="0.0"/>
+  <xacro:property name="namespace" value="$(arg namespace)"/>
+  <xacro:property name="x" value="$(arg x)"/>
+  <xacro:property name="y" value="$(arg y)"/>
+  <xacro:property name="z" value="$(arg z)"/>
   <xacro:property name="mode" value="differential" />
   <xacro:include filename="$(find minipock_description)/urdf/minipock_base.xacro" />
-  <xacro:minipock_base namespace="${namespace}" name="minipock" />
+  <xacro:minipock_base namespace="${namespace}" name="minipock" x="${x}" y="${y}" z="${z}"/>
   <!-- motor -->
   <xacro:include filename="$(find minipock_description)/urdf/motor.xacro" />
@@ -35,7 +42,8 @@
         <wheel_radius>0.036</wheel_radius>
         <odom_publish_frequency>50</odom_publish_frequency>
-        <topic>cmd_vel</topic>
-        <child_frame_id>${namespace}base_link</child_frame_id>
-        <frame_id>odom</frame_id>
+        <topic>${namespace}cmd_vel</topic>
+      <odom_topic>${namespace}odom</odom_topic>
+        <child_frame_id>${namespace}base_footprint</child_frame_id>
+        <frame_id>${namespace}odom</frame_id>
       </plugin>
     </xacro:if>

File: minipock_description/urdf/minipock_base.xacro (robot description, xacro)
@@ -1,5 +1,7 @@
 <?xml version="1.0"?>
 <robot name="minipock" xmlns:xacro="http://ros.org/wiki/xacro">
-  <xacro:macro name="minipock_base" params="namespace:=minipock name:=minipock">
+  <xacro:macro name="minipock_base" params="namespace:=minipock/ name:=minipock x:=0 y:=0 z:=0.0">
+    <link name="${namespace}base_footprint">
+    </link>
     <link name="${namespace}base_link">
       <visual>
@@ -21,5 +23,5 @@
       </inertial>
     </link>
-    <link name="${name}_structure_pla_link">
+    <link name="${namespace}minipock_structure_pla_link">
       <visual>
         <origin xyz="0 0 0.0" rpy="0 0 0" />
@@ -32,5 +34,5 @@
       </visual>
     </link>
-    <link name="${name}_structure_pmma_link">
+    <link name="${namespace}minipock_structure_pmma_link">
       <visual>
         <origin xyz="0 0 0.0" rpy="0 0 0" />
@@ -43,5 +45,5 @@
       </visual>
     </link>
-    <link name="${name}_structure_misc_link">
+    <link name="${namespace}minipock_structure_misc_link">
       <visual>
         <origin xyz="0 0 0.0" rpy="0 0 0" />
@@ -54,18 +56,23 @@
       </visual>
     </link>
-    <joint name="${name}_structure_pla_joint" type="fixed">
-      <origin xyz="0 0 0.0" rpy="0 0 ${-pi/2}" />
-      <parent link="${namespace}base_link" />
-      <child link="${name}_structure_pla_link" />
+    <joint name="base_joint" type="fixed">
+      <origin xyz="${x} ${y} ${z}" rpy="0 0 0"/>
+      <parent link="${namespace}base_footprint"/>
+      <child link="${namespace}base_link"/>
     </joint>
-    <joint name="${name}_structure_pmma_joint" type="fixed">
-      <origin xyz="0 0 0.0" rpy="0 0 ${-pi/2}" />
-      <parent link="${namespace}base_link" />
-      <child link="${name}_structure_pmma_link" />
+    <joint name="minipock_structure_pla_joint" type="fixed">
+      <origin xyz="0 0 0.0" rpy="0 0 ${-pi/2}"/>
+      <parent link="${namespace}base_link"/>
+      <child link="${namespace}minipock_structure_pla_link"/>
     </joint>
-    <joint name="${name}_structure_misc_joint" type="fixed">
-      <origin xyz="0 0 0.0" rpy="0 0 ${-pi/2}" />
-      <parent link="${namespace}base_link" />
-      <child link="${name}_structure_misc_link" />
+    <joint name="minipock_structure_pmma_joint" type="fixed">
+      <origin xyz="0 0 0.0" rpy="0 0 ${-pi/2}"/>
+      <parent link="${namespace}base_link"/>
+      <child link="${namespace}minipock_structure_pmma_link"/>
+    </joint>
+    <joint name="minipock_structure_misc_joint" type="fixed">
+      <origin xyz="0 0 0.0" rpy="0 0 ${-pi/2}"/>
+      <parent link="${namespace}base_link"/>
+      <child link="${namespace}minipock_structure_misc_link"/>
     </joint>
   </xacro:macro>

File: minipock_description/urdf/sensors.xacro (robot description, xacro)
@@ -1,6 +1,7 @@
-<robot xmlns:xacro="http://ros.org/wiki/xacro">
+<?xml version="1.0"?>
+<robot name="minipock" xmlns:xacro="http://ros.org/wiki/xacro">
   <xacro:macro name="lds_01"
-               params="namespace:=minipock name:=lds_01 x:=0.0 y:=0.0 z:=0.0 R:=0.0 P:=0.0 Y:=0.0">
-    <link name="${name}_link">
+              params="namespace:=minipock/ name:=lds_01 x:=0.0 y:=0.0 z:=0.0 R:=0.0 P:=0.0 Y:=0.0">
+    <link name="${namespace}${name}_link">
       <visual name="${name}_visual">
         <origin xyz="0 0 0" rpy="${pi/2} 0 0"/>
@@ -25,10 +26,10 @@
       <origin xyz="${x} ${y} ${z}" rpy="${R} ${P} ${Y}"/>
       <parent link="${namespace}base_link"/>
-      <child link="${name}_link"/>
+      <child link="${namespace}${name}_link"/>
     </joint>
-    <gazebo reference="${name}_link">
+    <gazebo reference="${namespace}${name}_link">
       <sensor type="gpu_lidar" name="lds_01">
         <update_rate>50</update_rate>
-        <topic>scan_raw</topic>
+        <topic>${namespace}scan_raw</topic>
         <visualize>true</visualize>
         <lidar>

Commit message: feat: Add namespace and update link names in minipock description

File: minipock_description/urdf/minipock.urdf.xacro (robot description, xacro)
@@ -1,7 +1,14 @@
 <?xml version="1.0"?>
 <robot name="minipock" xmlns:xacro="http://ros.org/wiki/xacro">
-  <xacro:property name="namespace" value="" />
+  <xacro:arg name="namespace" default="minipock/"/>
+  <xacro:arg name="x" default="0.0"/>
+  <xacro:arg name="y" default="0.0"/>
+  <xacro:arg name="z" default="0.0"/>
+  <xacro:property name="namespace" value="$(arg namespace)"/>
+  <xacro:property name="x" value="$(arg x)"/>
+  <xacro:property name="y" value="$(arg y)"/>
+  <xacro:property name="z" value="$(arg z)"/>
   <xacro:include filename="$(find minipock_description)/urdf/minipock_differential_base.xacro" />
-  <xacro:minipock_base namespace="${namespace}" name="minipock" />
+  <xacro:minipock_base namespace="${namespace}" name="minipock" x="${x}" y="${y}" z="${z}"/>
   <!-- motor -->
   <xacro:include filename="$(find minipock_description)/urdf/motor_stepper.xacro" />
@@ -25,7 +32,8 @@
       <wheel_radius>0.036</wheel_radius>
       <odom_publish_frequency>50</odom_publish_frequency>
-      <topic>cmd_vel</topic>
-      <child_frame_id>${namespace}base_link</child_frame_id>
-      <frame_id>odom</frame_id>
+      <topic>${namespace}cmd_vel</topic>
+      <odom_topic>${namespace}odom</odom_topic>
+      <child_frame_id>${namespace}base_footprint</child_frame_id>
+      <frame_id>${namespace}odom</frame_id>
     </plugin>
     <plugin filename="libgz-sim-pose-publisher-system.so"

File: minipock_description/urdf/minipock_differential_base.xacro (robot description, xacro)
@@ -1,5 +1,7 @@
 <?xml version="1.0"?>
 <robot name="minipock" xmlns:xacro="http://ros.org/wiki/xacro">
-  <xacro:macro name="minipock_base" params="namespace:=minipock name:=minipock">
+  <xacro:macro name="minipock_base" params="namespace:=minipock/ name:=minipock x:=0 y:=0 z:=0.0">
+    <link name="${namespace}base_footprint">
+    </link>
     <link name="${namespace}base_link">
       <visual>
@@ -21,5 +23,5 @@
       </inertial>
     </link>
-    <link name="${name}_structure_pla_link">
+    <link name="${namespace}minipock_structure_pla_link">
       <visual>
         <origin xyz="0 0 0.0" rpy="0 0 0" />
@@ -32,5 +34,5 @@
       </visual>
     </link>
-    <link name="${name}_structure_pmma_link">
+    <link name="${namespace}minipock_structure_pmma_link">
       <visual>
         <origin xyz="0 0 0.0" rpy="0 0 0" />
@@ -43,5 +45,5 @@
       </visual>
     </link>
-    <link name="${name}_structure_misc_link">
+    <link name="${namespace}minipock_structure_misc_link">
       <visual>
         <origin xyz="0 0 0.0" rpy="0 0 0" />
@@ -54,18 +56,23 @@
       </visual>
     </link>
-    <joint name="${name}_structure_pla_joint" type="fixed">
-      <origin xyz="0 0 0.0" rpy="0 0 ${-pi/2}" />
-      <parent link="${namespace}base_link" />
-      <child link="${name}_structure_pla_link" />
+    <joint name="base_joint" type="fixed">
+      <origin xyz="${x} ${y} ${z}" rpy="0 0 0"/>
+      <parent link="${namespace}base_footprint"/>
+      <child link="${namespace}base_link"/>
     </joint>
-    <joint name="${name}_structure_pmma_joint" type="fixed">
-      <origin xyz="0 0 0.0" rpy="0 0 ${-pi/2}" />
-      <parent link="${namespace}base_link" />
-      <child link="${name}_structure_pmma_link" />
+    <joint name="minipock_structure_pla_joint" type="fixed">
+      <origin xyz="0 0 0.0" rpy="0 0 ${-pi/2}"/>
+      <parent link="${namespace}base_link"/>
+      <child link="${namespace}minipock_structure_pla_link"/>
     </joint>
-    <joint name="${name}_structure_misc_joint" type="fixed">
-      <origin xyz="0 0 0.0" rpy="0 0 ${-pi/2}" />
-      <parent link="${namespace}base_link" />
-      <child link="${name}_structure_misc_link" />
+    <joint name="minipock_structure_pmma_joint" type="fixed">
+      <origin xyz="0 0 0.0" rpy="0 0 ${-pi/2}"/>
+      <parent link="${namespace}base_link"/>
+      <child link="${namespace}minipock_structure_pmma_link"/>
+    </joint>
+    <joint name="minipock_structure_misc_joint" type="fixed">
+      <origin xyz="0 0 0.0" rpy="0 0 ${-pi/2}"/>
+      <parent link="${namespace}base_link"/>
+      <child link="${namespace}minipock_structure_misc_link"/>
     </joint>
   </xacro:macro>

File: minipock_description/urdf/motor_stepper.xacro (robot description, xacro)
@@ -2,7 +2,7 @@
 <robot name="minipock" xmlns:xacro="http://ros.org/wiki/xacro">
   <xacro:macro name="motor_stepper"
-    params="namespace:=minipock name:=stepper_left x:=0.0 y:=0.0 z:=0.0
+    params="namespace:=minipock/ name:=stepper_left x:=0.0 y:=0.0 z:=0.0
 				       R:=0.0 P:=0.0 Y:=0.0 side:=1">
-    <link name="${name}_base_link">
+    <link name="${namespace}${name}_base_link">
       <visual>
         <origin xyz="0 0 0.0" rpy="${pi/2} 0 0" />
@@ -17,5 +17,5 @@
       </inertial>
     </link>
-    <link name="${name}_wheel_link">
+    <link name="${namespace}${name}_wheel_link">
       <visual>
         <origin xyz="0 0 -0.024" rpy="${pi/2} 0 0" />
@@ -38,10 +38,10 @@
     <joint name="${name}_joint" type="fixed">
       <parent link="${namespace}base_link" />
-      <child link="${name}_base_link" />
+      <child link="${namespace}${name}_base_link" />
       <origin xyz="${x} ${y} ${z}" rpy="${R} ${P} ${Y}" />
     </joint>
     <joint name="${name}_wheel_joint" type="continuous">
-      <parent link="${name}_base_link" />
-      <child link="${name}_wheel_link" />
+      <parent link="${namespace}${name}_base_link" />
+      <child link="${namespace}${name}_wheel_link" />
       <origin xyz="0.0 0.0 0.024" rpy="0 0 0" />
       <axis xyz="0 ${side} 0" />
