Commit message: refactor: Update minipock.urdf.xacro to use namespace variable for left and right joint names

File: minipock_description/urdf/minipock.urdf.xacro (robot description, xacro)
@@ -37,11 +37,11 @@
         filename="gz-sim-diff-drive-system"
         name="gz::sim::systems::DiffDrive">
-        <left_joint>motor_left_wheel_joint</left_joint>
-        <right_joint>motor_right_wheel_joint</right_joint>
+        <left_joint>${namespace}motor_left_wheel_joint</left_joint>
+        <right_joint>${namespace}motor_right_wheel_joint</right_joint>
         <wheel_separation>0.335</wheel_separation>
         <wheel_radius>0.036</wheel_radius>
         <odom_publish_frequency>50</odom_publish_frequency>
         <topic>${namespace}cmd_vel</topic>
-      <odom_topic>${namespace}odom</odom_topic>
+        <odom_topic>${namespace}odom</odom_topic>
         <child_frame_id>${namespace}base_footprint</child_frame_id>
         <frame_id>${namespace}odom</frame_id>

File: minipock_description/urdf/motor.xacro (robot description, xacro)
@@ -2,7 +2,7 @@
 <robot name="minipock" xmlns:xacro="http://ros.org/wiki/xacro">
   <xacro:macro name="motor"
-    params="namespace:=minipock name:=motor_left x:=0.0 y:=0.0 z:=0.0
+    params="namespace:=minipock/ name:=motor_left x:=0.0 y:=0.0 z:=0.0
 				       R:=0.0 P:=0.0 Y:=0.0 side:=1 mode:='differential'">
-    <link name="${name}_base_link">
+    <link name="${namespace}${name}_base_link">
       <visual>
         <origin xyz="0 0 0.0" rpy="${pi/2} 0 0" />
@@ -18,5 +18,5 @@
     </link>
     <xacro:if value="${mode == 'differential'}">
-      <link name="${name}_wheel_link">
+      <link name="${namespace}${name}_wheel_link">
         <visual>
           <origin xyz="0 0 -0.024" rpy="${pi/2} 0 0" />
@@ -37,7 +37,7 @@
         </inertial>
       </link>
-      <joint name="${name}_wheel_joint" type="continuous">
-        <parent link="${name}_base_link" />
-        <child link="${name}_wheel_link" />
+      <joint name="${namespace}${name}_wheel_joint" type="continuous">
+        <parent link="${namespace}${name}_base_link" />
+        <child link="${namespace}${name}_wheel_link" />
         <origin xyz="0.0 0.0 0.024" rpy="0 0 0" />
         <axis xyz="0 ${side} 0" />
@@ -46,5 +46,5 @@
     </xacro:if>
     <xacro:if value="${mode == 'holonomic'}">
-      <link name="${name}_wheel_link">
+      <link name="${namespace}${name}_wheel_link">
         <visual>
           <origin xyz="-4.8572257327350598644e-17 0 -0.0099999999999999793915"
@@ -53,5 +53,5 @@
             <mesh filename="package://minipock_description/models/wheel_core.stl" />
           </geometry>
-          <material name="${name}_wheel_link_material">
+          <material name="${namespace}${name}_wheel_link_material">
             <color
               rgba="0.06862745098039220171 0.08627450980392152857 0.05294117647058818044 1.0" />
@@ -68,12 +68,12 @@
         </inertial>
       </link>
-      <joint name="${name}_wheel_joint" type="continuous">
-        <parent link="${name}_base_link" />
-        <child link="${name}_wheel_link" />
+      <joint name="${namespace}${name}_wheel_joint" type="continuous">
+        <parent link="${namespace}${name}_base_link" />
+        <child link="${namespace}${name}_wheel_link" />
         <origin xyz="0.0 0.02 0.024" rpy="${pi/2} 0 0" />
         <axis xyz="0 0 ${side}" />
         <limit effort="2000" velocity="45.5" />
       </joint>
-      <link name="${name}_roller">
+      <link name="${namespace}${name}_roller">
         <visual>
           <origin xyz="0 3.4694469519536141888e-18 -0.0080000000000000019013"
@@ -104,13 +104,13 @@
         </inertial>
       </link>
-      <joint name="${name}_joint_roller_6_continuous" type="continuous">
+      <joint name="${namespace}${name}_joint_roller_6_continuous" type="continuous">
         <origin xyz="-0.028131604665040808172 0.013220856400772910966 -0.0049999999999999905631"
           rpy="-1.3962634015950849964 1.5707963267948952257 0" />
-        <parent link="${name}_wheel_link" />
-        <child link="${name}_roller" />
-        <axis xyz="0 0 1" />
-         <limit effort="1" velocity="200" />
-      </joint>
-      <link name="${name}_roller_2">
+        <parent link="${namespace}${name}_wheel_link" />
+        <child link="${namespace}${name}_roller" />
+        <axis xyz="0 0 1" />
+         <limit effort="1" velocity="200" />
+      </joint>
+      <link name="${namespace}${name}_roller_2">
         <visual>
           <origin xyz="0 0 -0.0080000000000000001665"
@@ -141,13 +141,13 @@
         </inertial>
       </link>
-      <joint name="${name}_joint_roller_5_continuous" type="continuous">
+      <joint name="${namespace}${name}_joint_roller_5_continuous" type="continuous">
         <origin xyz="-0.030048262113536068629 -0.0079548833402023552686 -0.0049999999999999801548"
           rpy="-2.0943951023928160105 1.5707963267948950037 0" />
-        <parent link="${name}_wheel_link" />
-        <child link="${name}_roller_2" />
-        <axis xyz="0 0 1" />
-         <limit effort="1" velocity="200" />
-      </joint>
-      <link name="${name}_roller_3">
+        <parent link="${namespace}${name}_wheel_link" />
+        <child link="${namespace}${name}_roller_2" />
+        <axis xyz="0 0 1" />
+         <limit effort="1" velocity="200" />
+      </joint>
+      <link name="${namespace}${name}_roller_3">
         <visual>
           <origin xyz="0 -6.9388939039072283776e-18 -0.008000000000000003636"
@@ -178,13 +178,13 @@
         </inertial>
       </link>
-      <joint name="${name}_joint_roller_4_continuous" type="continuous">
+      <joint name="${namespace}${name}_joint_roller_4_continuous" type="continuous">
         <origin xyz="-0.017905003769872984004 -0.025408444757616242826 -0.0049999999999999775527"
           rpy="-2.7925268031905519095 1.5707963267948958919 0" />
-        <parent link="${name}_wheel_link" />
-        <child link="${name}_roller_3" />
-        <axis xyz="0 0 1" />
-         <limit effort="1" velocity="200" />
-      </joint>
-      <link name="${name}_roller_4">
+        <parent link="${namespace}${name}_wheel_link" />
+        <child link="${namespace}${name}_roller_3" />
+        <axis xyz="0 0 1" />
+         <limit effort="1" velocity="200" />
+      </joint>
+      <link name="${namespace}${name}_roller_4">
         <visual>
           <origin xyz="0 3.4694469519536141888e-18 -0.0079999999999999984318"
@@ -215,13 +215,13 @@
         </inertial>
       </link>
-      <joint name="${name}_joint_roller_3_continuous" type="continuous">
+      <joint name="${namespace}${name}_joint_roller_3_continuous" type="continuous">
         <origin xyz="0.0026162048296650758025 -0.030973112489532557412 -0.0049999999999999723485"
           rpy="2.7925268031913015321 1.5707963267948958919 0" />
-        <parent link="${name}_wheel_link" />
-        <child link="${name}_roller_4" />
-        <axis xyz="0 0 1" />
-         <limit effort="1" velocity="200" />
-      </joint>
-      <link name="${name}_roller_5">
+        <parent link="${namespace}${name}_wheel_link" />
+        <child link="${namespace}${name}_roller_4" />
+        <axis xyz="0 0 1" />
+         <limit effort="1" velocity="200" />
+      </joint>
+      <link name="${namespace}${name}_roller_5">
         <visual>
           <origin xyz="0 0 -0.0080000000000000001665"
@@ -252,13 +252,13 @@
         </inertial>
       </link>
-      <joint name="${name}_joint_roller_2_continuous" type="continuous">
+      <joint name="${namespace}${name}_joint_roller_2_continuous" type="continuous">
         <origin xyz="0.021913262113524886732 -0.022045116659794552344 -0.0049999999999999723485"
           rpy="2.0943951023935678535 1.5707963267948958919 0" />
-        <parent link="${name}_wheel_link" />
-        <child link="${name}_roller_5" />
-        <axis xyz="0 0 1" />
-         <limit effort="1" velocity="200" />
-      </joint>
-      <link name="${name}_roller_6">
+        <parent link="${namespace}${name}_wheel_link" />
+        <child link="${namespace}${name}_roller_5" />
+        <axis xyz="0 0 1" />
+         <limit effort="1" velocity="200" />
+      </joint>
+      <link name="${namespace}${name}_roller_6">
         <visual>
           <origin xyz="0 0 -0.0080000000000000019013"
@@ -289,13 +289,13 @@
         </inertial>
       </link>
-      <joint name="${name}_joint_roller_1_continuous" type="continuous">
+      <joint name="${namespace}${name}_joint_roller_1_continuous" type="continuous">
         <origin xyz="0.030956860515685625385 -0.002801965740757847434 -0.0049999999999999801548"
           rpy="1.3962634015958343969 1.5707963267948956698 0" />
-        <parent link="${name}_wheel_link" />
-        <child link="${name}_roller_6" />
-        <axis xyz="0 0 1" />
-         <limit effort="1" velocity="200" />
-      </joint>
-      <link name="${name}_roller_7">
+        <parent link="${namespace}${name}_wheel_link" />
+        <child link="${namespace}${name}_roller_6" />
+        <axis xyz="0 0 1" />
+         <limit effort="1" velocity="200" />
+      </joint>
+      <link name="${namespace}${name}_roller_7">
         <visual>
           <origin
@@ -328,13 +328,13 @@
         </inertial>
       </link>
-      <joint name="${name}_joint_roller_9_continuous" type="continuous">
+      <joint name="${namespace}${name}_joint_roller_9_continuous" type="continuous">
         <origin xyz="0.025515399835375589255 0.017752256088759903185 -0.004999999999999987961"
           rpy="0.69813170079810316082 1.5707963267948954478 0" />
-        <parent link="${name}_wheel_link" />
-        <child link="${name}_roller_7" />
-        <axis xyz="0 0 1" />
-         <limit effort="1" velocity="200" />
-      </joint>
-      <link name="${name}_roller_8">
+        <parent link="${namespace}${name}_wheel_link" />
+        <child link="${namespace}${name}_roller_7" />
+        <axis xyz="0 0 1" />
+         <limit effort="1" velocity="200" />
+      </joint>
+      <link name="${namespace}${name}_roller_8">
         <visual>
           <origin xyz="0 0 -0.0080000000000000001665"
@@ -365,13 +365,13 @@
         </inertial>
       </link>
-      <joint name="${name}_joint_roller_8_continuous" type="continuous">
+      <joint name="${namespace}${name}_joint_roller_8_continuous" type="continuous">
         <origin xyz="0.0081350000000113779214 0.029999999999996886796 -0.0049999999999999792874"
           rpy="3.8172294696792983199e-13 1.570796326794896558 0" />
-        <parent link="${name}_wheel_link" />
-        <child link="${name}_roller_8" />
-        <axis xyz="0 0 1" />
-         <limit effort="1" velocity="200" />
-      </joint>
-      <link name="${name}_roller_9">
+        <parent link="${namespace}${name}_wheel_link" />
+        <child link="${namespace}${name}_roller_8" />
+        <axis xyz="0 0 1" />
+         <limit effort="1" velocity="200" />
+      </joint>
+      <link name="${namespace}${name}_roller_9">
         <visual>
           <origin xyz="0 0 -0.0080000000000000001665"
@@ -402,9 +402,9 @@
         </inertial>
       </link>
-      <joint name="${name}_joint_roller_7_continuous" type="continuous">
+      <joint name="${namespace}${name}_joint_roller_7_continuous" type="continuous">
         <origin xyz="-0.013258688745465072728 0.028036857843754141306 -0.0049999999999999992367"
           rpy="-0.69813170079771968979 1.5707963267948958919 0" />
-        <parent link="${name}_wheel_link" />
-        <child link="${name}_roller_9" />
+        <parent link="${namespace}${name}_wheel_link" />
+        <child link="${namespace}${name}_roller_9" />
         <axis xyz="0 0 1" />
          <limit effort="1" velocity="200" />
@@ -412,7 +412,7 @@
       </joint>
     </xacro:if>
-    <joint name="${name}_joint" type="fixed">
+    <joint name="${namespace}${name}_joint" type="fixed">
       <parent link="${namespace}base_link" />
-      <child link="${name}_base_link" />
+      <child link="${namespace}${name}_base_link" />
       <origin xyz="${x} ${y} ${z}" rpy="${R} ${P} ${Y}" />
     </joint>
@@ -421,5 +421,5 @@
         name="gz::sim::systems::JointController">
         <joint_name>${name}_wheel_joint</joint_name>
-        <use_velocity_commands>false</use_velocity_commands>
+        <use_velocity_commands>true</use_velocity_commands>
         <topic>${namespace}${name}/pos</topic>
         <name>${name}</name>

Commit message: refactor: Update xacro_cmd function to accept mode parameter for holonomic or differential mode

File: minipock_description/urdf/minipock.urdf.xacro (robot description, xacro)
@@ -5,9 +5,10 @@
   <xacro:arg name="y" default="0.0"/>
   <xacro:arg name="z" default="0.0"/>
+  <xacro:arg name="mode" default="differential"/>
   <xacro:property name="namespace" value="$(arg namespace)"/>
   <xacro:property name="x" value="$(arg x)"/>
   <xacro:property name="y" value="$(arg y)"/>
   <xacro:property name="z" value="$(arg z)"/>
-  <xacro:property name="mode" value="differential" />
+  <xacro:property name="mode" value="$(arg mode)"/>
   <xacro:include filename="$(find minipock_description)/urdf/minipock_base.xacro" />
   <xacro:minipock_base namespace="${namespace}" name="minipock" x="${x}" y="${y}" z="${z}"/>

Commit message: Refactor: rename lidar references from lds_01 to lidar in URDF and RViz files

File: minipock_description/urdf/minipock.urdf.xacro (robot description, xacro)
@@ -31,5 +31,5 @@
   <!-- sensors -->
   <xacro:include filename="$(find minipock_description)/urdf/sensors.xacro" />
-  <xacro:lds_01 namespace="${namespace}" name="lds_01" x="0.0" y="0.0" z="0.050" R="${pi}" P="0.0"
+  <xacro:lidar namespace="${namespace}" name="lidar" x="0.0" y="0.0" z="0.050" R="${pi}" P="0.0"
     Y="0.0" />
   <gazebo>

File: minipock_description/urdf/minipock_base.xacro (robot description, xacro)
@@ -14,5 +14,5 @@
         <origin xyz="0 0 -${0.089/2}" rpy="0 -0 ${-pi/2}" />
         <geometry>
-          <cylinder radius="0.15" length="0.092" />
+          <cylinder radius="0.15" length="0.098" />
         </geometry>
       </collision>

File: minipock_description/urdf/sensors.xacro (robot description, xacro)
@@ -1,6 +1,6 @@
 <?xml version="1.0"?>
 <robot name="minipock" xmlns:xacro="http://ros.org/wiki/xacro">
-  <xacro:macro name="lds_01"
-              params="namespace:=minipock/ name:=lds_01 x:=0.0 y:=0.0 z:=0.0 R:=0.0 P:=0.0 Y:=0.0">
+  <xacro:macro name="lidar"
+              params="namespace:=minipock/ name:=lidar x:=0.0 y:=0.0 z:=0.0 R:=0.0 P:=0.0 Y:=0.0">
     <link name="${namespace}${name}_link">
       <visual name="${name}_visual">
@@ -29,5 +29,5 @@
     </joint>
     <gazebo reference="${namespace}${name}_link">
-      <sensor type="gpu_lidar" name="lds_01">
+      <sensor type="gpu_lidar" name="lidar">
         <update_rate>10</update_rate>
         <topic>${namespace}scan_raw</topic>
